Commit message: sensors parent

File: rmodus_sim/urdf/bumpers.urdf.xacro (robot description, xacro)
@@ -4,5 +4,4 @@
 <!-- PROPERTY -->
 <xacro:property name='bumper_mass'      value='0.01'/>
-<xacro:property name='bumper_parent' default='base_link'/>
 <!-- BUMPERS -->
 <gazebo>
@@ -24,5 +23,5 @@
   </link>
   <joint name="bumper_${b['name']}_joint" type="fixed">
-    <parent link="${bumper_parent}"/>
+    <parent link="${b['parent_frame']}"/>
     <child link="bumper_${b['name']}_link"/>
     <origin xyz="${b['offset'][0]} ${b['offset'][1]} ${b['offset'][2]}"

File: rmodus_sim/urdf/cliff_sensors.urdf.xacro (robot description, xacro)
@@ -4,5 +4,4 @@
 <!-- PROPERTY -->
 <xacro:property name='cliff_sensor_mass' value='0.001'/>
-<xacro:property name='cliff_sensor_parent' default='base_link'/>
 <!-- CLIFF_SENSORS -->
 <xacro:macro name="render_cliff_sensor" params="c">
@@ -19,5 +18,5 @@
   </link>
   <joint name="cliff_sensor_${c['name']}_joint" type="fixed">
-    <parent link="${cliff_sensor_parent}"/>
+    <parent link="${b['parent_frame']}"/>
     <child link="cliff_sensor_${c['name']}_link"/>
     <origin xyz="${c['offset'][0]} ${c['offset'][1]} ${c['offset'][2]}"
