Commit message: websocket-sensors

File: rmodus_sim/urdf/cliff_sensors.urdf.xacro (robot description, xacro)
@@ -18,5 +18,5 @@
   </link>
   <joint name="cliff_sensor_${c['name']}_joint" type="fixed">
-    <parent link="${b['parent_frame']}"/>
+    <parent link="${c['parent_frame']}"/>
     <child link="cliff_sensor_${c['name']}_link"/>
     <origin xyz="${c['offset'][0]} ${c['offset'][1]} ${c['offset'][2]}"
