Commit message: rmodus_description

File: rmodus_sim/urdf/robot.urdf.xacro (robot description, xacro)
@@ -1,3 +1,5 @@
 <?xml version='1.0'?>
+<!-- Simulation robot description.
+     Includes the shared base from rmodus_description and adds Gazebo plugins. -->
 <robot
   name='my_robot'
@@ -5,19 +7,22 @@
   xmlns:gz='http://gazebosim.org/schema'>
 <!-- ARGUMENTS -->
-<xacro:arg name="config_path" default="" />
-<!-- CONFIG -->
-<xacro:property name="robot_cfg" value="${xacro.load_yaml('$(arg config_path)')}" />
-<xacro:property name="bumpers" value="${robot_cfg['/**']['ros__parameters']['bumpers']}" />
-<xacro:property name="cliff_sensors" value="${robot_cfg['/**']['ros__parameters']['cliff_sensors']}" />
-<!-- CONSTANTS -->
+<xacro:arg name='config_path' default='' />
+<!-- CONSTANTS used by sim-specific xacro (mesh paths) -->
 <xacro:property name='meshes_dir' value='rmodus_sim/meshes'/>
 <xacro:property name='creo_scale' value='0.001' />
-<!-- COLORS -->
-<xacro:property name='alpha' value='1'/> <!-- {0 - 1} -->
+<!-- Shared config and helpers -->
+<xacro:property name='robot_cfg' value="${xacro.load_yaml('$(arg config_path)')}" />
+<xacro:property name='bumpers' value="${robot_cfg['/**']['ros__parameters']['bumpers']}" />
+<xacro:property name='cliff_sensors' value="${robot_cfg['/**']['ros__parameters']['cliff_sensors']}" />
+<xacro:property name='base_cfg' value="${robot_cfg['/**']['ros__parameters']['base_link']}" />
+<xacro:property name='imu_cfg' value="${robot_cfg['/**']['ros__parameters']['imu']}" />
+<xacro:property name='lidar_cfg' value="${robot_cfg['/**']['ros__parameters']['lidar']}" />
+<xacro:property name='use_mesh' value='true' />
+<xacro:property name='mesh_scale' value='${creo_scale}' />
+<xacro:property name='alpha' value='1'/>
 <material name='red'> <color rgba='0.8 0.0 0.0 ${alpha}'/> </material>
 <material name='green'> <color rgba='0.0 0.8 0.0 ${alpha}'/> </material>
 <material name='blue'> <color rgba='0.0 0.0 0.8 ${alpha}'/> </material>
 <material name='gray'> <color rgba='0.5 0.5 0.5 ${alpha}'/> </material>
-<!-- FUNCTIONS -->
 <xacro:macro name='box_inertia' params='m x y z'>
   <inertial>
@@ -32,7 +37,7 @@
     <mass value='${m}'/>
     <inertia ixx='${m/12 * (3*r*r + h*h)}' ixy='0.0' ixz='0.0'
-              iyy='${m/12 * (3*r*r + h*h)}' iyz='0.0'
-              izz='${m/2 * r*r}'/>
-    </inertial>
+             iyy='${m/12 * (3*r*r + h*h)}' iyz='0.0'
+             izz='${m/2 * r*r}'/>
+  </inertial>
 </xacro:macro>
 <xacro:macro name='sphere_inertia' params='m r'>
@@ -44,11 +49,17 @@
   </inertial>
 </xacro:macro>
-<!-- INCLUDE -->
-<xacro:include filename='base.urdf.xacro'/>
-<xacro:include filename='bumpers.urdf.xacro'/>
-<xacro:include filename='cliff_sensors.urdf.xacro'/>
+<!-- Include shared base components -->
+<xacro:include filename='$(find rmodus_description)/urdf/base.urdf.xacro'/>
+<xacro:include filename='$(find rmodus_description)/urdf/imu.urdf.xacro'/>
+<xacro:include filename='$(find rmodus_description)/urdf/lidar.urdf.xacro'/>
+<xacro:include filename='$(find rmodus_description)/urdf/bumpers.urdf.xacro'/>
+<xacro:include filename='$(find rmodus_description)/urdf/cliff_sensors.urdf.xacro'/>
+<!-- Sim-only: wheels with mesh visuals -->
 <xacro:include filename='wheels.urdf.xacro'/>
-<xacro:include filename='lidar.urdf.xacro'/>
-<xacro:include filename='imu.urdf.xacro'/>
+<!-- Sim-only: Gazebo sensor plugins -->
+<xacro:include filename='gz_imu.urdf.xacro'/>
+<xacro:include filename='gz_lidar.urdf.xacro'/>
+<xacro:include filename='gz_bumpers.urdf.xacro'/>
+<xacro:include filename='gz_cliff_sensors.urdf.xacro'/>
 <xacro:include filename='control.urdf.xacro'/>
 </robot>
