Commit message: sim samostatnot

File: rmodus_sim/urdf/base.urdf.xacro (robot description, xacro)
@@ -1,28 +1,28 @@
-<?xml version="1.0"?>
-<robot xmlns:xacro='http://www.ros.org/wiki/xacro'
-       xmlns:gz='http://gazebosim.org/schema'>
-<!-- PROPERTY -->
-<xacro:property name='base_mass' value='5'/>
-<xacro:property name='base_size_x' value='0.3'/>
-<xacro:property name='base_size_y' value='0.3'/>
-<xacro:property name='base_size_z' value='0.1'/>
-<xacro:property name='base_offset_z' value='0.0973 '/> <!-- 0.0973 -->
-<xacro:property name='nav_offset_z' value='0'/>
-<xacro:property name='nav_offset_x' value='0.032'/>
-<!-- LINKS -->
-<link name='base_footprint'>
-</link>
+<?xml version='1.0'?>
+<!-- Local sim base structure used when structure_source is local. -->
+<robot xmlns:xacro='http://www.ros.org/wiki/xacro'>
+<xacro:property name='base_mass'     value='${base_cfg["mass"]}'/>
+<xacro:property name='base_size_x'   value='${base_cfg["size"][0]}'/>
+<xacro:property name='base_size_y'   value='${base_cfg["size"][1]}'/>
+<xacro:property name='base_size_z'   value='${base_cfg["size"][2]}'/>
+<xacro:property name='base_offset_z' value='${base_cfg["offset_z"]}'/>
+<xacro:property name='nav_offset_x'  value='${base_cfg["nav_offset_x"]}'/>
+<xacro:property name='nav_offset_z'  value='${base_cfg["nav_offset_z"]}'/>
+<link name='base_footprint'/>
 <link name='base_link'>
   <xacro:box_inertia m='${base_mass}' x='${base_size_x}' y='${base_size_y}' z='${base_size_z}'/>
   <visual>
-    <geometry>
-      <mesh filename='package://${meshes_dir}/base.obj' scale='${creo_scale} ${creo_scale} ${creo_scale}'/>
-    </geometry>
+    <xacro:if value='${use_mesh == "true"}'>
+      <geometry>
+        <mesh filename='package://${meshes_dir}/base.obj' scale='${mesh_scale} ${mesh_scale} ${mesh_scale}'/>
+      </geometry>
+    </xacro:if>
+    <xacro:unless value='${use_mesh == "true"}'>
+      <geometry><box size='${base_size_x} ${base_size_y} ${base_size_z}'/></geometry>
+    </xacro:unless>
     <material name='blue'/>
   </visual>
   <collision>
-    <geometry>
-      <box size='${base_size_x} ${base_size_y} ${base_size_z}'/>
-    </geometry>
+    <geometry><box size='${base_size_x} ${base_size_y} ${base_size_z}'/></geometry>
   </collision>
 </link>
@@ -30,13 +30,19 @@
   <visual>
     <origin xyz='0 0 0' rpy='0 0 0'/>
-    <geometry> <mesh filename='package://${meshes_dir}/navigation.obj' scale='${creo_scale} ${creo_scale} ${creo_scale}'/> </geometry>
+    <xacro:if value='${use_mesh == "true"}'>
+      <geometry>
+        <mesh filename='package://${meshes_dir}/navigation.obj' scale='${mesh_scale} ${mesh_scale} ${mesh_scale}'/>
+      </geometry>
+    </xacro:if>
+    <xacro:unless value='${use_mesh == "true"}'>
+      <geometry><cylinder radius='0.01' length='0.04'/></geometry>
+    </xacro:unless>
     <material name='gray'/>
   </visual>
 </link>
-<!-- JOINTS -->
 <joint name='body_link_joint' type='fixed'>
-    <parent link='base_footprint' />
-    <child link='base_link' />
-    <origin xyz='0 0 ${base_offset_z}' rpy='0 0 0'/>
+  <parent link='base_footprint'/>
+  <child link='base_link'/>
+  <origin xyz='0 0 ${base_offset_z}' rpy='0 0 0'/>
 </joint>
 <joint name='nav_module_mount_joint' type='fixed'>

File: rmodus_sim/urdf/bumpers.urdf.xacro (robot description, xacro)
@@ -1,67 +1,32 @@
-<?xml version="1.0"?>
-<robot xmlns:xacro='http://www.ros.org/wiki/xacro'
-       xmlns:gz='http://gazebosim.org/schema'>
-<!-- PROPERTY -->
-<xacro:property name='bumper_mass'      value='0.01'/>
-<!-- BUMPERS -->
-<gazebo>
-  <plugin filename="libgz-sim-contact-system.so" name="gz::sim::systems::Contact" />
-</gazebo>
-<xacro:macro name="render_bumper" params="b">
-  <!-- Bumper link -->
-  <link name="bumper_${b['name']}_link">
-    <xacro:box_inertia m="${bumper_mass}" x="${b['size'][0]}" y="${b['size'][1]}" z="${b['size'][2]}"/>
+<?xml version='1.0'?>
+<!-- Local sim bumper TF frames used when structure_source is local. -->
+<robot xmlns:xacro='http://www.ros.org/wiki/xacro'>
+<xacro:property name='bumper_mass' value='0.01'/>
+<xacro:macro name='render_bumper' params='b'>
+  <link name='bumper_${b["name"]}_link'>
+    <xacro:box_inertia m='${bumper_mass}' x='${b["size"][0]}' y='${b["size"][1]}' z='${b["size"][2]}'/>
     <visual>
-      <origin xyz="${b['size'][0]/2} 0 0" rpy="0 0 0"/>
-      <geometry><box size="${b['size'][0]} ${b['size'][1]} ${b['size'][2]}"/></geometry>
-      <material name="red"/>
+      <origin xyz='${b["size"][0]/2} 0 0' rpy='0 0 0'/>
+      <geometry><box size='${b["size"][0]} ${b["size"][1]} ${b["size"][2]}'/></geometry>
+      <material name='red'/>
     </visual>
     <collision>
-      <origin xyz="${b['size'][0]/2} 0 0" rpy="0 0 0"/>
-      <geometry><box size="${b['size'][0]} ${b['size'][1]} ${b['size'][2]}"/></geometry>
+      <origin xyz='${b["size"][0]/2} 0 0' rpy='0 0 0'/>
+      <geometry><box size='${b["size"][0]} ${b["size"][1]} ${b["size"][2]}'/></geometry>
     </collision>
   </link>
-  <joint name="bumper_${b['name']}_joint" type="fixed">
-    <parent link="${b['parent_frame']}"/>
-    <child link="bumper_${b['name']}_link"/>
-    <origin xyz="${b['offset'][0]} ${b['offset'][1]} ${b['offset'][2]}"
-            rpy="0 0 ${b['yaw']}"/>
+  <joint name='bumper_${b["name"]}_joint' type='fixed'>
+    <parent link='${b["parent_frame"]}'/>
+    <child link='bumper_${b["name"]}_link'/>
+    <origin xyz='${b["offset"][0]} ${b["offset"][1]} ${b["offset"][2]}' rpy='0 0 ${b["yaw"]}'/>
   </joint>
-  <gazebo reference="bumper_${b['name']}_joint">
-    <preserveFixedJoint>true</preserveFixedJoint>
-  </gazebo>
-  <gazebo reference="bumper_${b['name']}_link">
-    <sensor name="bumper_${b['name']}_sensor" type="contact">
-      <always_on>1</always_on>
-      <update_rate>30</update_rate>
-      <topic>/bumper/${b['name']}</topic>
-      <contact>
-        <collision>bumper_${b['name']}_link_collision</collision>
-      </contact>
-    </sensor>
-  </gazebo>
-  <!-- Contact frame -->
-  <link name="bumper_${b['name']}_contact_frame">
-    <inertial>
-      <mass value="0.001"/> <inertia ixx="0.00001" ixy="0" ixz="0" iyy="0.00001" iyz="0" izz="0.00001"/>
-    </inertial>
-  </link>
-  <joint name="bumper_${b['name']}_contact_joint" type="fixed">
-    <parent link="bumper_${b['name']}_link"/>
-    <child link="bumper_${b['name']}_contact_frame"/>
-    <origin xyz="${b['size'][0]} 0 0" rpy="0 0 0"/>
-  </joint>
-  <gazebo reference="bumper_${b['name']}_contact_joint">
-    <preserveFixedJoint>true</preserveFixedJoint>
-  </gazebo>
 </xacro:macro>
-<xacro:macro name="bumper_loop" params="items">
-  <xacro:if value="${items}">
-    <xacro:property name="current_b" value="${items.pop(0)}"/>
-    <xacro:render_bumper b="${current_b}" />
-    <xacro:bumper_loop items="${items}"/>
+<xacro:macro name='bumper_loop' params='items'>
+  <xacro:if value='${items}'>
+    <xacro:property name='current_b' value='${items.pop(0)}'/>
+    <xacro:render_bumper b='${current_b}'/>
+    <xacro:bumper_loop items='${items}'/>
   </xacro:if>
 </xacro:macro>
-<xacro:bumper_loop items="${list(bumpers)}"/>
-<!-- /BUMPERS -->
+<xacro:bumper_loop items='${list(bumpers)}'/>
 </robot>

File: rmodus_sim/urdf/cliff_sensors.urdf.xacro (robot description, xacro)
@@ -1,76 +1,38 @@
-<?xml version="1.0"?>
-<robot xmlns:xacro='http://www.ros.org/wiki/xacro'
-       xmlns:gz='http://gazebosim.org/schema'>
-<!-- PROPERTY -->
+<?xml version='1.0'?>
+<!-- Local sim cliff TF frames used when structure_source is local. -->
+<robot xmlns:xacro='http://www.ros.org/wiki/xacro'>
 <xacro:property name='cliff_sensor_mass' value='0.001'/>
-<!-- CLIFF_SENSORS -->
-<xacro:macro name="render_cliff_sensor" params="c">
-  <!-- Sensor link -->
-  <link name="cliff_sensor_${c['name']}_link">
-    <xacro:box_inertia m="${cliff_sensor_mass}" x="${c['size'][0]}" y="${c['size'][1]}" z="${c['size'][2]}"/>
+<xacro:macro name='render_cliff_sensor' params='c'>
+  <link name='cliff_sensor_${c["name"]}_link'>
+    <xacro:box_inertia m='${cliff_sensor_mass}' x='${c["size"][0]}' y='${c["size"][1]}' z='${c["size"][2]}'/>
     <visual>
-      <geometry><box size="${c['size'][0]} ${c['size'][1]} ${c['size'][2]}"/></geometry>
-      <material name="red"/>
+      <geometry><box size='${c["size"][0]} ${c["size"][1]} ${c["size"][2]}'/></geometry>
+      <material name='red'/>
     </visual>
-    <!-- <collision>
-      <geometry><box size="${c['size'][0]} ${c['size'][1]} ${c['size'][2]}"/></geometry>
-    </collision> -->
   </link>
-  <joint name="cliff_sensor_${c['name']}_joint" type="fixed">
-    <parent link="${c['parent_frame']}"/>
-    <child link="cliff_sensor_${c['name']}_link"/>
-    <origin xyz="${c['offset'][0]} ${c['offset'][1]} ${c['offset'][2]}"
-            rpy="0 0 ${c.get('yaw', 0.0)}"/>
+  <joint name='cliff_sensor_${c["name"]}_joint' type='fixed'>
+    <parent link='${c["parent_frame"]}'/>
+    <child link='cliff_sensor_${c["name"]}_link'/>
+    <origin xyz='${c["offset"][0]} ${c["offset"][1]} ${c["offset"][2]}' rpy='0 0 ${c.get("yaw", 0.0)}'/>
   </joint>
-  <gazebo reference="cliff_sensor_${c['name']}_link">
-    <preserveFixedJoint>true</preserveFixedJoint>
-  </gazebo>
-  <!-- Beam frame -->
-  <link name="cliff_sensor_${c['name']}_beam_frame">
+  <link name='cliff_sensor_${c["name"]}_beam_frame'>
     <inertial>
-      <mass value="0.001"/> <inertia ixx="0.00001" ixy="0" ixz="0" iyy="0.00001" iyz="0" izz="0.00001"/>
+      <mass value='0.001'/>
+      <inertia ixx='0.00001' ixy='0' ixz='0' iyy='0.00001' iyz='0' izz='0.00001'/>
     </inertial>
   </link>
-  <joint name="cliff_sensor_${c['name']}_beam_joint" type="fixed">
-    <parent link="cliff_sensor_${c['name']}_link"/>
-    <child link="cliff_sensor_${c['name']}_beam_frame"/>
-    <origin xyz="0 0 ${-c['size'][2]/2}" rpy="0 ${pi/2} 0"/>
+  <joint name='cliff_sensor_${c["name"]}_beam_joint' type='fixed'>
+    <parent link='cliff_sensor_${c["name"]}_link'/>
+    <child link='cliff_sensor_${c["name"]}_beam_frame'/>
+    <origin xyz='0 0 ${-c["size"][2]/2}' rpy='0 ${pi/2} 0'/>
   </joint>
-  <gazebo reference="cliff_sensor_${c['name']}_beam_joint">
-    <preserveFixedJoint>true</preserveFixedJoint>
-  </gazebo>
-  <gazebo reference="cliff_sensor_${c['name']}_beam_frame">
-    <sensor name="cliff_${c['name']}" type="gpu_ray">
-      <always_on>1</always_on>
-      <update_rate>20</update_rate>
-      <visualize>true</visualize>
-      <ray>
-        <scan>
-          <horizontal>
-            <samples>1</samples>
-            <resolution>1</resolution>
-            <min_angle>0</min_angle>
-            <max_angle>0</max_angle>
-          </horizontal>
-        </scan>
-        <range>
-          <min>0.01</min>
-          <max>0.5</max>
-          <resolution>0.001</resolution>
-        </range>
-      </ray>
-      <topic>/cliff/${c['name']}</topic>
-      <gz_frame_id>cliff_sensor_${c['name']}_beam_frame</gz_frame_id>
-    </sensor>
-  </gazebo>
 </xacro:macro>
-<xacro:macro name="cliff_sensor_loop" params="items">
-  <xacro:if value="${items}">
-    <xacro:property name="current_c" value="${items.pop(0)}"/>
-    <xacro:render_cliff_sensor c="${current_c}" />
-    <xacro:cliff_sensor_loop items="${items}"/>
+<xacro:macro name='cliff_sensor_loop' params='items'>
+  <xacro:if value='${items}'>
+    <xacro:property name='current_c' value='${items.pop(0)}'/>
+    <xacro:render_cliff_sensor c='${current_c}'/>
+    <xacro:cliff_sensor_loop items='${items}'/>
   </xacro:if>
 </xacro:macro>
-<xacro:cliff_sensor_loop items="${list(cliff_sensors)}"/>
-<!-- /CLIFF_SENSORS -->
+<xacro:cliff_sensor_loop items='${list(cliff_sensors)}'/>
 </robot>

File: rmodus_sim/urdf/gz_bumpers.urdf.xacro (robot description, xacro)
@@ -9,4 +9,5 @@
 </gazebo>
 <xacro:macro name='gz_bumper_sensors' params='b'>
+  <xacro:if value='${b.get("enabled", True)}'>
   <gazebo reference='bumper_${b["name"]}_joint'>
     <preserveFixedJoint>true</preserveFixedJoint>
@@ -15,6 +16,6 @@
     <sensor name='bumper_${b["name"]}_sensor' type='contact'>
       <always_on>1</always_on>
-      <update_rate>30</update_rate>
-      <topic>/bumper/${b["name"]}</topic>
+      <update_rate>${b.get("update_rate", 30)}</update_rate>
+      <topic>${b.get("topic", "/bumper/" + b["name"])}</topic>
       <contact>
         <collision>bumper_${b["name"]}_link_collision</collision>
@@ -37,4 +38,5 @@
     <preserveFixedJoint>true</preserveFixedJoint>
   </gazebo>
+  </xacro:if>
 </xacro:macro>
 <xacro:macro name='gz_bumper_loop' params='items'>

File: rmodus_sim/urdf/gz_cliff_sensors.urdf.xacro (robot description, xacro)
@@ -5,4 +5,5 @@
        xmlns:gz='http://gazebosim.org/schema'>
 <xacro:macro name='gz_cliff_sensor' params='c'>
+  <xacro:if value='${c.get("enabled", True)}'>
   <gazebo reference='cliff_sensor_${c["name"]}_link'>
     <preserveFixedJoint>true</preserveFixedJoint>
@@ -14,6 +15,6 @@
     <sensor name='cliff_${c["name"]}' type='gpu_ray'>
       <always_on>1</always_on>
-      <update_rate>20</update_rate>
-      <visualize>true</visualize>
+      <update_rate>${c.get("update_rate", 20)}</update_rate>
+      <visualize>${str(c.get("visualize", True)).lower()}</visualize>
       <ray>
         <scan>
@@ -26,13 +27,14 @@
         </scan>
         <range>
-          <min>0.01</min>
-          <max>0.5</max>
-          <resolution>0.001</resolution>
+          <min>${c.get("range_min", 0.01)}</min>
+          <max>${c.get("range_max", 0.5)}</max>
+          <resolution>${c.get("range_resolution", 0.001)}</resolution>
         </range>
       </ray>
-      <topic>/cliff/${c["name"]}</topic>
+      <topic>${c.get("topic", "/cliff/" + c["name"])}</topic>
       <gz_frame_id>cliff_sensor_${c["name"]}_beam_frame</gz_frame_id>
     </sensor>
   </gazebo>
+  </xacro:if>
 </xacro:macro>
 <xacro:macro name='gz_cliff_sensor_loop' params='items'>

File: rmodus_sim/urdf/gz_imu.urdf.xacro (robot description, xacro)
@@ -13,7 +13,7 @@
   <sensor name='imu_sensor' type='imu'>
     <always_on>1</always_on>
-    <update_rate>100</update_rate>
-    <visualize>false</visualize>
-    <topic>imu/data</topic>
+    <update_rate>${imu_cfg.get("update_rate", 100)}</update_rate>
+    <visualize>${str(imu_cfg.get("visualize", False)).lower()}</visualize>
+    <topic>${imu_cfg.get("topic", "/imu/data")}</topic>
     <imu>
       <angular_velocity>

File: rmodus_sim/urdf/gz_lidar.urdf.xacro (robot description, xacro)
@@ -14,21 +14,21 @@
   <sensor name='lidar' type='gpu_ray'>
     <always_on>1</always_on>
-    <visualize>false</visualize>
-    <update_rate>10</update_rate>
+    <visualize>${str(lidar_cfg.get("visualize", False)).lower()}</visualize>
+    <update_rate>${lidar_cfg.get("update_rate", 10)}</update_rate>
     <ray>
       <scan>
         <horizontal>
-          <samples>360</samples>
+          <samples>${max(1, int(round(lidar_cfg.get("fov", 360) / max(lidar_cfg.get("resolution", 1.0), 1e-6))))}</samples>
           <resolution>1.0</resolution>
-          <min_angle>0.0</min_angle>
-          <max_angle>${2*pi}</max_angle>
+          <min_angle>${lidar_cfg.get("angle_min", 0.0)}</min_angle>
+          <max_angle>${lidar_cfg.get("angle_max", 2 * pi)}</max_angle>
         </horizontal>
       </scan>
       <range>
-        <min>0.05</min>
-        <max>5.0</max>
+        <min>${lidar_cfg.get("range_min", 0.05)}</min>
+        <max>${lidar_cfg.get("range_max", 5.0)}</max>
       </range>
     </ray>
-    <topic>scan</topic>
+    <topic>${lidar_cfg.get("topic", "/scan")}</topic>
     <gz_frame_id>lidar_beam</gz_frame_id>
   </sensor>

File: rmodus_sim/urdf/imu.urdf.xacro (robot description, xacro)
@@ -1,9 +1,8 @@
-<?xml version="1.0"?>
-<robot xmlns:xacro='http://www.ros.org/wiki/xacro'
-       xmlns:gz='http://gazebosim.org/schema'>
-<!-- IMU -->
+<?xml version='1.0'?>
+<!-- Local sim IMU TF frame used when structure_source is local. -->
+<robot xmlns:xacro='http://www.ros.org/wiki/xacro'>
 <link name='imu_mount'>
   <visual>
-    <geometry> <box size='0.02 0.02 0.01'/> </geometry>
+    <geometry><box size='0.02 0.02 0.01'/></geometry>
     <material name='red'/>
   </visual>
@@ -14,26 +13,3 @@
   <origin xyz='${imu_cfg["offset_x"]} ${imu_cfg["offset_y"]} ${imu_cfg["offset_z"]}' rpy='0 0 0'/>
 </joint>
-<gazebo>
-  <plugin
-    filename='libgz-sim-imu-system.so'
-    name='gz::sim::systems::Imu'>
-  </plugin>
-</gazebo>
-<gazebo reference='imu_mount'>
-  <sensor name='imu_sensor' type='imu'>
-    <always_on>1</always_on>
-    <update_rate>100</update_rate>
-    <visualize>false</visualize>
-    <topic>imu/data</topic>
-    <imu>
-      <angular_velocity>
-        <x><noise type='gaussian'><mean>0.0</mean><stddev>1e-4</stddev></noise></x>
-      </angular_velocity>
-      <linear_acceleration>
-        <x><noise type='gaussian'><mean>0.0</mean><stddev>1e-3</stddev></noise></x>
-      </linear_acceleration>
-    </imu>
-  </sensor>
-</gazebo>
-<!-- /IMU -->
 </robot>

File: rmodus_sim/urdf/lidar.urdf.xacro (robot description, xacro)
@@ -1,9 +1,8 @@
-<?xml version="1.0"?>
-<robot xmlns:xacro='http://www.ros.org/wiki/xacro'
-       xmlns:gz='http://gazebosim.org/schema'>
-<!-- LIDAR -->
+<?xml version='1.0'?>
+<!-- Local sim lidar TF frame used when structure_source is local. -->
+<robot xmlns:xacro='http://www.ros.org/wiki/xacro'>
 <link name='lidar_beam'>
   <visual>
-    <geometry> <cylinder radius='0.01' length='0.04'/> </geometry>
+    <geometry><cylinder radius='0.01' length='0.04'/></geometry>
     <material name='red'/>
   </visual>
@@ -14,34 +13,3 @@
   <origin xyz='${lidar_cfg["offset_x"]} 0 ${lidar_cfg["offset_z"]}' rpy='0 0 0'/>
 </joint>
-<gazebo>
-  <plugin
-    filename='libgz-sim-sensors-system.so'
-    name='gz::sim::systems::Sensors'>
-    <render_engine>ogre2</render_engine>
-  </plugin>
-</gazebo>
-<gazebo reference='lidar_beam'>
-  <sensor name='lidar' type='gpu_ray'>
-    <always_on>1</always_on>
-    <visualize>false</visualize>
-    <update_rate>10</update_rate>
-    <ray>
-      <scan>
-        <horizontal>
-          <samples>360</samples>
-          <resolution>1.0</resolution>
-          <min_angle>0.0</min_angle>
-          <max_angle>${2*pi}</max_angle>
-        </horizontal>
-      </scan>
-      <range>
-        <min>0.05</min>
-        <max>5.0</max>
-      </range>
-    </ray>
-    <topic>scan</topic>
-    <gz_frame_id>lidar_beam</gz_frame_id>
-  </sensor>
-</gazebo>
-<!-- /LIDAR -->
 </robot>

File: rmodus_sim/urdf/robot.urdf.xacro (robot description, xacro)
@@ -8,4 +8,6 @@
 <!-- ARGUMENTS -->
 <xacro:arg name='config_path' default='' />
+<xacro:arg name='structure_source' default='local' />
+<xacro:property name='structure_source' value='$(arg structure_source)'/>
 <!-- CONSTANTS used by sim-specific xacro (mesh paths) -->
 <xacro:property name='meshes_dir' value='rmodus_sim/meshes'/>
@@ -49,10 +51,19 @@
   </inertial>
 </xacro:macro>
-<!-- Include shared base components -->
-<xacro:include filename='$(find rmodus_description)/urdf/base.urdf.xacro'/>
-<xacro:include filename='$(find rmodus_description)/urdf/imu.urdf.xacro'/>
-<xacro:include filename='$(find rmodus_description)/urdf/lidar.urdf.xacro'/>
-<xacro:include filename='$(find rmodus_description)/urdf/bumpers.urdf.xacro'/>
-<xacro:include filename='$(find rmodus_description)/urdf/cliff_sensors.urdf.xacro'/>
+<!-- Structural components are switchable by source. -->
+<xacro:if value='${structure_source == "description"}'>
+  <xacro:include filename='$(find rmodus_description)/urdf/base.urdf.xacro'/>
+  <xacro:include filename='$(find rmodus_description)/urdf/imu.urdf.xacro'/>
+  <xacro:include filename='$(find rmodus_description)/urdf/lidar.urdf.xacro'/>
+  <xacro:include filename='$(find rmodus_description)/urdf/bumpers.urdf.xacro'/>
+  <xacro:include filename='$(find rmodus_description)/urdf/cliff_sensors.urdf.xacro'/>
+</xacro:if>
+<xacro:unless value='${structure_source == "description"}'>
+  <xacro:include filename='base.urdf.xacro'/>
+  <xacro:include filename='imu.urdf.xacro'/>
+  <xacro:include filename='lidar.urdf.xacro'/>
+  <xacro:include filename='bumpers.urdf.xacro'/>
+  <xacro:include filename='cliff_sensors.urdf.xacro'/>
+</xacro:unless>
 <!-- Sim-only: wheels with mesh visuals -->
 <xacro:include filename='wheels.urdf.xacro'/>
