Commit message: multiple bumpers+cliff

File: rmodus_hw/urdf/robot.urdf.xacro (robot description, xacro)
@@ -7,11 +7,10 @@
   xmlns:xacro='http://www.ros.org/wiki/xacro'
   xmlns:gz='http://gazebosim.org/schema'>
-<!-- CONFIGURABLE SENSOR GEOMETRY -->
-<xacro:arg name='lidar_offset_z' default='0.2'/>
-<xacro:arg name='lidar_offset_x' default='0.005'/>
-<xacro:arg name='imu_offset_z'   default='0.015'/>
-<xacro:arg name='imu_offset_x'   default='0.056'/>
-<xacro:arg name='imu_offset_y'   default='0.020'/>
-<xacro:arg name='cliff_sensor_z' default='-0.02'/>
+<!-- ARGUMENTS -->
+<xacro:arg name="config_path" default="" />
+<!-- CONFIG -->
+<xacro:property name="robot_cfg" value="${xacro.load_yaml('$(arg config_path)')}" />
+<xacro:property name="bumpers" value="${robot_cfg['/**']['ros__parameters']['bumpers']}" />
+<xacro:property name="cliff_sensors" value="${robot_cfg['/**']['ros__parameters']['cliff_sensors']}" />
 <!-- CONSTANTS -->
 <xacro:property name='base_mass' value='5'/>
@@ -27,4 +26,11 @@
 <xacro:property name='bumper_height'    value='0.04'/>
 <xacro:property name='bumper_mass'      value='0.01'/>
+<xacro:arg name='lidar_offset_z' default='0.2'/>
+<xacro:arg name='lidar_offset_x' default='0.005'/>
+<xacro:arg name='imu_offset_z'   default='0.015'/>
+<xacro:arg name='imu_offset_x'   default='0.056'/>
+<xacro:arg name='imu_offset_y'   default='0.020'/>
+<xacro:arg name='cliff_sensor_z' default='-0.02'/>
+<xacro:arg name='bumper_parent' default='base_link'/>
 <!-- COLORS -->
 <xacro:property name='alpha' value='1'/> <!-- {0 - 1} -->
@@ -68,17 +74,21 @@
   </link>
 </xacro:macro>
-<!-- MACRO: Bumper panel link (with collision for contact detection) -->
-<xacro:macro name='bumper_link' params='name len_x len_y'>
-  <link name='bumper_${name}_link'>
-    <xacro:box_inertia m='${bumper_mass}' x='${len_x}' y='${len_y}' z='${bumper_height}'/>
+<!-- BUMPERS -->
+<xacro:foreach items="${bumpers}" name="b">
+  <link name="bumper_${b['name']}_link">
+    <xacro:box_inertia m="${bumper_mass}" x="${b['depth']}" y="${b['width']}" z="${b['height']}"/>
     <visual>
-      <geometry><box size='${len_x} ${len_y} ${bumper_height}'/></geometry>
-      <material name='red'/>
+      <geometry><box size="${b['depth']} ${b['width']} ${b['height']}"/></geometry>
+      <material name="red"/>
     </visual>
-    <collision name='bumper_${name}_link'>
-      <geometry><box size='${len_x} ${len_y} ${bumper_height}'/></geometry>
-    </collision>
   </link>
-</xacro:macro>
+  <joint name="bumper_${b['name']}_joint" type="fixed">
+    <parent link="$(arg bumper_parent)"/>
+    <child link="bumper_${b['name']}_link"/>
+    <origin xyz="${b['offset'][0]} ${b['offset'][1]} ${b['offset'][2]}"
+            rpy="${b['rotation'][0]} ${b['rotation'][1]} ${b['rotation'][2]}"/>
+  </joint>
+</xacro:foreach>
+<!-- /BUMPERS -->
 <!-- LINKS -->
 <link name='base_footprint'>
@@ -122,9 +132,4 @@
 <xacro:cliff_sensor_link name='cliff_rl'/>
 <xacro:cliff_sensor_link name='cliff_rr'/>
-<!-- BUMPER LINKS (4 strany) -->
-<xacro:bumper_link name='front' len_x='${bumper_thickness}' len_y='${base_size_y}'/>
-<xacro:bumper_link name='rear'  len_x='${bumper_thickness}' len_y='${base_size_y}'/>
-<xacro:bumper_link name='left'  len_x='${base_size_x}'      len_y='${bumper_thickness}'/>
-<xacro:bumper_link name='right' len_x='${base_size_x}'      len_y='${bumper_thickness}'/>
 <!-- JOINTS -->
 <joint name='body_link_joint' type='fixed'>

File: rmodus_sim/urdf/robot.urdf.xacro (robot description, xacro)
@@ -2,36 +2,15 @@
 <robot
   name='my_robot'
-  xmlns:xacro='http://www.ros.org/wiki/xacro'
+  xmlns:xacro='http://ros.org/wiki/xacro'
   xmlns:gz='http://gazebosim.org/schema'>
+<!-- ARGUMENTS -->
+<xacro:arg name="config_path" default="" />
+<!-- CONFIG -->
+<xacro:property name="robot_cfg" value="${xacro.load_yaml('$(arg config_path)')}" />
+<xacro:property name="bumpers" value="${robot_cfg['/**']['ros__parameters']['bumpers']}" />
+<xacro:property name="cliff_sensors" value="${robot_cfg['/**']['ros__parameters']['cliff_sensors']}" />
 <!-- CONSTANTS -->
-<!-- mecanum dont publish odom topic in Gazebo 8.9.0 !!!, use 8.10.0 instead or diff-->
-<xacro:property name='drive' value='mecanum'/> <!-- mecanum or diff -->
 <xacro:property name='meshes_dir' value='rmodus_sim/meshes'/>
 <xacro:property name='creo_scale' value='0.001' />
-<xacro:property name='base_mass' value='5'/>
-<xacro:property name='base_size_x' value='0.5'/>
-<xacro:property name='base_size_y' value='0.5'/>
-<xacro:property name='base_size_z' value='0.1'/>
-<xacro:property name='wheel_mass' value='0.5'/>
-<xacro:property name='wheelbase' value='0.179'/>
-<xacro:property name='track_width' value='0.327'/>
-<xacro:property name='wheel_radius' value='0.05'/>
-<xacro:property name='wheel_length' value='0.03'/>
-<xacro:property name='wheel_mu' value='1.0'/>
-<xacro:property name='wheel_mu2' value='0.1'/>
-<xacro:property name='base_offset_z' value='0.0973 '/> <!-- 0.0973 -->
-<xacro:property name='wheel_offset_z' value='-0.0473'/>
-<xacro:property name='nav_offset_z' value='0'/>
-<xacro:property name='nav_offset_x' value='0.032'/>
-<xacro:property name='lidar_offset_z' value='0.2'/>
-<xacro:property name='lidar_offset_x' value='0.005'/>
-<xacro:property name='imu_offset_z' value='0.015'/>
-<xacro:property name='imu_offset_x' value='0.056'/>
-<xacro:property name='imu_offset_y' value='0.020'/>
-<xacro:property name='cliff_sensor_z'    value='-0.02'/>
-<xacro:property name='cliff_sensor_mass' value='0.001'/>
-<xacro:property name='bumper_thickness' value='0.005'/>
-<xacro:property name='bumper_height'    value='0.04'/>
-<xacro:property name='bumper_mass'      value='0.01'/>
 <!-- COLORS -->
 <xacro:property name='alpha' value='1'/> <!-- {0 - 1} -->
@@ -65,219 +44,11 @@
   </inertial>
 </xacro:macro>
-<!-- MACRO: Cliff sensor link (visual only, fixed joint) -->
-<xacro:macro name='cliff_sensor_link' params='name'>
-  <link name='${name}_link'>
-    <xacro:box_inertia m='${cliff_sensor_mass}' x='0.015' y='0.015' z='0.02'/>
-    <visual>
-      <geometry><box size='0.015 0.015 0.02'/></geometry>
-      <material name='red'/>
-    </visual>
-  </link>
-</xacro:macro>
-<!-- MACRO: Bumper panel link (with collision for contact detection) -->
-<xacro:macro name='bumper_link' params='name len_x len_y'>
-  <link name='bumper_${name}_link'>
-    <xacro:box_inertia m='${bumper_mass}' x='${len_x}' y='${len_y}' z='${bumper_height}'/>
-    <visual>
-      <geometry><box size='${len_x} ${len_y} ${bumper_height}'/></geometry>
-      <material name='red'/>
-    </visual>
-    <collision name='bumper_${name}_link'>
-      <geometry><box size='${len_x} ${len_y} ${bumper_height}'/></geometry>
-    </collision>
-  </link>
-</xacro:macro>
-<!-- LINKS -->
-<link name='base_footprint'>
-</link>
-<link name='base_link'>
-  <xacro:box_inertia m='${base_mass}' x='${base_size_x}' y='${base_size_y}' z='${base_size_z}'/>
-  <visual>
-    <geometry>
-      <mesh filename='package://${meshes_dir}/base.obj' scale='${creo_scale} ${creo_scale} ${creo_scale}'/>
-    </geometry>
-    <material name='blue'/>
-  </visual>
-  <collision>
-    <geometry>
-      <box size='${base_size_x} ${base_size_y} ${base_size_z}'/>
-    </geometry>
-  </collision>
-</link>
-<link name='front_left_wheel'>
-  <xacro:sphere_inertia m='${wheel_mass}' r='${wheel_radius}' />
-  <visual>
-    <geometry>
-      <mesh filename='package://${meshes_dir}/wheel.obj' scale='${creo_scale} ${creo_scale} ${creo_scale}'/>
-    </geometry>
-    <material name='green'/>
-  </visual>
-  <collision>
-    <geometry>
-      <sphere radius='${wheel_radius}'/>
-    </geometry>
-  </collision>
-</link>
-<link name='front_right_wheel'>
-  <xacro:sphere_inertia m='${wheel_mass}' r='${wheel_radius}' />
-  <visual>
-    <origin xyz='0 0 0' rpy='0 ${pi} 0'/>
-    <geometry>
-      <mesh filename='package://${meshes_dir}/wheel_mirror.obj' scale='${creo_scale} ${creo_scale} ${creo_scale}'/>
-    </geometry>
-    <material name='green'/>
-  </visual>
-  <collision>
-    <geometry>
-      <sphere radius='${wheel_radius}'/>
-    </geometry>
-  </collision>
-</link>
-<link name='rear_left_wheel'>
-  <xacro:sphere_inertia m='${wheel_mass}' r='${wheel_radius}' />
-  <visual>
-    <geometry>
-      <mesh filename='package://${meshes_dir}/wheel_mirror.obj' scale='${creo_scale} ${creo_scale} ${creo_scale}'/>
-    </geometry>
-    <material name='green'/>
-  </visual>
-  <collision>
-    <geometry>
-      <sphere radius='${wheel_radius}'/>
-    </geometry>
-  </collision>
-</link>
-<link name='rear_right_wheel'>
-  <xacro:sphere_inertia m='${wheel_mass}' r='${wheel_radius}' />
-  <visual>
-    <origin xyz='0 0 0' rpy='0 ${pi} 0'/>
-    <geometry>
-      <mesh filename='package://${meshes_dir}/wheel.obj' scale='${creo_scale} ${creo_scale} ${creo_scale}'/>
-    </geometry>
-    <material name='green'/>
-  </visual>
-  <collision>
-    <geometry>
-      <sphere radius='${wheel_radius}'/>
-    </geometry>
-  </collision>
-</link>
-<link name='nav_module_mount'>
-  <visual>
-    <origin xyz='0 0 0' rpy='0 0 0'/>
-    <geometry> <mesh filename='package://${meshes_dir}/navigation.obj' scale='${creo_scale} ${creo_scale} ${creo_scale}'/> </geometry>
-    <material name='gray'/>
-  </visual>
-</link>
-<link name='lidar_beam'>
-  <visual>
-    <geometry> <cylinder radius='0.01' length='0.04'/> </geometry>
-    <material name='red'/>
-  </visual>
-</link>
-<link name='imu_mount'>
-  <visual>
-    <geometry> <box size='0.02 0.02 0.01'/> </geometry>
-    <material name='red'/>
-  </visual>
-</link>
-<!-- CLIFF SENSOR LINKS (4 rohy) -->
-<xacro:cliff_sensor_link name='cliff_fl'/>
-<xacro:cliff_sensor_link name='cliff_fr'/>
-<xacro:cliff_sensor_link name='cliff_rl'/>
-<xacro:cliff_sensor_link name='cliff_rr'/>
-<!-- BUMPER LINKS (4 strany) -->
-<xacro:bumper_link name='front' len_x='${bumper_thickness}' len_y='${base_size_y}'/>
-<xacro:bumper_link name='rear'  len_x='${bumper_thickness}' len_y='${base_size_y}'/>
-<xacro:bumper_link name='left'  len_x='${base_size_x}'      len_y='${bumper_thickness}'/>
-<xacro:bumper_link name='right' len_x='${base_size_x}'      len_y='${bumper_thickness}'/>
-<!-- JOINTS -->
-<joint name='body_link_joint' type='fixed'>
-    <parent link='base_footprint' />
-    <child link='base_link' />
-    <origin xyz='0 0 ${base_offset_z}' rpy='0 0 0'/>
-</joint>
-<joint name='front_left_wheel_joint' type='continuous'>
-  <parent link='base_link'/>
-  <child link='front_left_wheel'/>
-  <origin xyz='${wheelbase/2} ${track_width/2} ${wheel_offset_z}' rpy='${-pi/2} 0 0'/>
-  <axis xyz='0 0 1'/>
-</joint>
-<joint name='front_right_wheel_joint' type='continuous'>
-  <parent link='base_link'/>
-  <child link='front_right_wheel'/>
-  <origin xyz='${wheelbase/2} ${-track_width/2} ${wheel_offset_z}' rpy='${-pi/2} 0 0'/>
-  <axis xyz='0 0 1'/>
-</joint>
-<joint name='rear_left_wheel_joint' type='continuous'>
-  <parent link='base_link'/>
-  <child link='rear_left_wheel'/>
-  <origin xyz='${-wheelbase/2} ${track_width/2} ${wheel_offset_z}' rpy='${-pi/2} 0 0'/>
-  <axis xyz='0 0 1'/>
-</joint>
-<joint name='rear_right_wheel_joint' type='continuous'>
-  <parent link='base_link'/>
-  <child link='rear_right_wheel'/>
-  <origin xyz='${-wheelbase/2} ${-track_width/2} ${wheel_offset_z}' rpy='${-pi/2} 0 0'/>
-  <axis xyz='0 0 1'/>
-</joint>
-<joint name='nav_module_mount_joint' type='fixed'>
-  <parent link='base_link'/>
-  <child link='nav_module_mount'/>
-  <origin xyz='${nav_offset_x} 0 ${nav_offset_z}' rpy='0 0 0'/>
-</joint>
-<joint name='lidar_joint' type='fixed'>
-  <parent link='nav_module_mount'/>
-  <child link='lidar_beam'/>
-  <origin xyz='${lidar_offset_x} 0 ${lidar_offset_z}' rpy='0 0 0'/>
-</joint>
-<joint name='imu_joint' type='fixed'>
-  <parent link='nav_module_mount'/>
-  <child link='imu_mount'/>
-  <origin xyz='${imu_offset_x} ${imu_offset_y} ${imu_offset_z}' rpy='0 0 0'/>
-</joint>
-<!-- CLIFF SENSOR JOINTS -->
-<joint name='cliff_fl_joint' type='fixed'>
-  <parent link='base_link'/>
-  <child link='cliff_fl_link'/>
-  <origin xyz='${base_size_x/2} ${base_size_y/2} ${cliff_sensor_z}' rpy='0 ${pi/2} 0'/>
-</joint>
-<joint name='cliff_fr_joint' type='fixed'>
-  <parent link='base_link'/>
-  <child link='cliff_fr_link'/>
-  <origin xyz='${base_size_x/2} ${-base_size_y/2} ${cliff_sensor_z}' rpy='0 ${pi/2} 0'/>
-</joint>
-<joint name='cliff_rl_joint' type='fixed'>
-  <parent link='base_link'/>
-  <child link='cliff_rl_link'/>
-  <origin xyz='${-base_size_x/2} ${base_size_y/2} ${cliff_sensor_z}' rpy='0 ${pi/2} 0'/>
-</joint>
-<joint name='cliff_rr_joint' type='fixed'>
-  <parent link='base_link'/>
-  <child link='cliff_rr_link'/>
-  <origin xyz='${-base_size_x/2} ${-base_size_y/2} ${cliff_sensor_z}' rpy='0 ${pi/2} 0'/>
-</joint>
-<!-- BUMPER JOINTS (strany, panel těsně vně těla robota) -->
-<joint name='bumper_front_joint' type='fixed'>
-  <parent link='base_link'/>
-  <child link='bumper_front_link'/>
-  <origin xyz='${base_size_x/2 + bumper_thickness/2} 0 0' rpy='0 0 0'/>
-</joint>
-<joint name='bumper_rear_joint' type='fixed'>
-  <parent link='base_link'/>
-  <child link='bumper_rear_link'/>
-  <origin xyz='${-(base_size_x/2 + bumper_thickness/2)} 0 0' rpy='0 0 0'/>
-</joint>
-<joint name='bumper_left_joint' type='fixed'>
-  <parent link='base_link'/>
-  <child link='bumper_left_link'/>
-  <origin xyz='0 ${base_size_y/2 + bumper_thickness/2} 0' rpy='0 0 0'/>
-</joint>
-<joint name='bumper_right_joint' type='fixed'>
-  <parent link='base_link'/>
-  <child link='bumper_right_link'/>
-  <origin xyz='0 ${-(base_size_y/2 + bumper_thickness/2)} 0' rpy='0 0 0'/>
-</joint>
-<!-- PLUGINS -->
-<xacro:include filename='robot.gazebo'/>
+<!-- INCLUDE -->
+<xacro:include filename='base.urdf.xacro'/>
+<xacro:include filename='bumpers.urdf.xacro'/>
+<xacro:include filename='cliff_sensors.urdf.xacro'/>
+<xacro:include filename='wheels.urdf.xacro'/>
+<xacro:include filename='lidar.urdf.xacro'/>
+<xacro:include filename='imu.urdf.xacro'/>
+<xacro:include filename='control.urdf.xacro'/>
 </robot>

Commit message: repair

File: rmodus_hw/urdf/robot.urdf.xacro (robot description, xacro)
@@ -64,31 +64,4 @@
   </inertial>
 </xacro:macro>
-<!-- MACRO: Cliff sensor link (visual only, fixed joint) -->
-<xacro:macro name='cliff_sensor_link' params='name'>
-  <link name='${name}_link'>
-    <xacro:box_inertia m='${cliff_sensor_mass}' x='0.015' y='0.015' z='0.02'/>
-    <visual>
-      <geometry><box size='0.015 0.015 0.02'/></geometry>
-      <material name='red'/>
-    </visual>
-  </link>
-</xacro:macro>
-<!-- BUMPERS -->
-<xacro:foreach items="${bumpers}" name="b">
-  <link name="bumper_${b['name']}_link">
-    <xacro:box_inertia m="${bumper_mass}" x="${b['depth']}" y="${b['width']}" z="${b['height']}"/>
-    <visual>
-      <geometry><box size="${b['depth']} ${b['width']} ${b['height']}"/></geometry>
-      <material name="red"/>
-    </visual>
-  </link>
-  <joint name="bumper_${b['name']}_joint" type="fixed">
-    <parent link="$(arg bumper_parent)"/>
-    <child link="bumper_${b['name']}_link"/>
-    <origin xyz="${b['offset'][0]} ${b['offset'][1]} ${b['offset'][2]}"
-            rpy="${b['rotation'][0]} ${b['rotation'][1]} ${b['rotation'][2]}"/>
-  </joint>
-</xacro:foreach>
-<!-- /BUMPERS -->
 <!-- LINKS -->
 <link name='base_footprint'>
@@ -153,45 +126,3 @@
   <origin xyz='$(arg imu_offset_x) $(arg imu_offset_y) $(arg imu_offset_z)' rpy='0 0 0'/>
 </joint>
-<!-- CLIFF SENSOR JOINTS -->
-<joint name='cliff_fl_joint' type='fixed'>
-  <parent link='base_link'/>
-  <child link='cliff_fl_link'/>
-  <origin xyz='${base_size_x/2} ${base_size_y/2} $(arg cliff_sensor_z)' rpy='0 ${pi/2} 0'/>
-</joint>
-<joint name='cliff_fr_joint' type='fixed'>
-  <parent link='base_link'/>
-  <child link='cliff_fr_link'/>
-  <origin xyz='${base_size_x/2} ${-base_size_y/2} $(arg cliff_sensor_z)' rpy='0 ${pi/2} 0'/>
-</joint>
-<joint name='cliff_rl_joint' type='fixed'>
-  <parent link='base_link'/>
-  <child link='cliff_rl_link'/>
-  <origin xyz='${-base_size_x/2} ${base_size_y/2} $(arg cliff_sensor_z)' rpy='0 ${pi/2} 0'/>
-</joint>
-<joint name='cliff_rr_joint' type='fixed'>
-  <parent link='base_link'/>
-  <child link='cliff_rr_link'/>
-  <origin xyz='${-base_size_x/2} ${-base_size_y/2} $(arg cliff_sensor_z)' rpy='0 ${pi/2} 0'/>
-</joint>
-<!-- BUMPER JOINTS (strany, panel těsně vně těla robota) -->
-<joint name='bumper_front_joint' type='fixed'>
-  <parent link='base_link'/>
-  <child link='bumper_front_link'/>
-  <origin xyz='${base_size_x/2 + bumper_thickness/2} 0 0' rpy='0 0 0'/>
-</joint>
-<joint name='bumper_rear_joint' type='fixed'>
-  <parent link='base_link'/>
-  <child link='bumper_rear_link'/>
-  <origin xyz='${-(base_size_x/2 + bumper_thickness/2)} 0 0' rpy='0 0 0'/>
-</joint>
-<joint name='bumper_left_joint' type='fixed'>
-  <parent link='base_link'/>
-  <child link='bumper_left_link'/>
-  <origin xyz='0 ${base_size_y/2 + bumper_thickness/2} 0' rpy='0 0 0'/>
-</joint>
-<joint name='bumper_right_joint' type='fixed'>
-  <parent link='base_link'/>
-  <child link='bumper_right_link'/>
-  <origin xyz='0 ${-(base_size_y/2 + bumper_thickness/2)} 0' rpy='0 0 0'/>
-</joint>
 </robot>

Commit message: rep

File: rmodus_hw/urdf/robot.urdf.xacro (robot description, xacro)
@@ -71,5 +71,5 @@
   <visual>
     <geometry>
-      <mesh filename='package://${meshes_dir}/base.obj' scale='${creo_scale} ${creo_scale} ${creo_scale}'/>
+      <box size='${base_size_x} ${base_size_y} ${base_size_z}'/>
     </geometry>
     <material name='blue'/>
@@ -84,5 +84,5 @@
   <visual>
     <origin xyz='0 0 0' rpy='0 0 0'/>
-    <geometry> <mesh filename='package://${meshes_dir}/navigation.obj' scale='${creo_scale} ${creo_scale} ${creo_scale}'/> </geometry>
+    <geometry> <cylinder radius='0.01' length='0.04'/> </geometry>
     <material name='gray'/>
   </visual>

Commit message: params

File: rmodus_hw/urdf/robot.urdf.xacro (robot description, xacro)
@@ -13,4 +13,6 @@
 <xacro:property name="bumpers" value="${robot_cfg['/**']['ros__parameters']['bumpers']}" />
 <xacro:property name="cliff_sensors" value="${robot_cfg['/**']['ros__parameters']['cliff_sensors']}" />
+<xacro:property name="imu_cfg" value="${robot_cfg['/**']['ros__parameters']['imu']}" />
+<xacro:property name="lidar_cfg" value="${robot_cfg['/**']['ros__parameters']['lidar']}" />
 <!-- CONSTANTS -->
 <xacro:property name='base_mass' value='5'/>
@@ -26,10 +28,4 @@
 <xacro:property name='bumper_height'    value='0.04'/>
 <xacro:property name='bumper_mass'      value='0.01'/>
-<xacro:arg name='lidar_offset_z' default='0.2'/>
-<xacro:arg name='lidar_offset_x' default='0.005'/>
-<xacro:arg name='imu_offset_z'   default='0.015'/>
-<xacro:arg name='imu_offset_x'   default='0.056'/>
-<xacro:arg name='imu_offset_y'   default='0.020'/>
-<xacro:arg name='cliff_sensor_z' default='-0.02'/>
 <xacro:arg name='bumper_parent' default='base_link'/>
 <!-- COLORS -->
@@ -114,10 +110,10 @@
   <parent link='nav_module_mount'/>
   <child link='lidar_beam'/>
-  <origin xyz='$(arg lidar_offset_x) 0 $(arg lidar_offset_z)' rpy='0 0 0'/>
+  <origin xyz='${lidar_cfg["offset_x"]} 0 ${lidar_cfg["offset_z"]}' rpy='0 0 0'/>
 </joint>
 <joint name='imu_joint' type='fixed'>
   <parent link='nav_module_mount'/>
   <child link='imu_mount'/>
-  <origin xyz='$(arg imu_offset_x) $(arg imu_offset_y) $(arg imu_offset_z)' rpy='0 0 0'/>
+  <origin xyz='${imu_cfg["offset_x"]} ${imu_cfg["offset_y"]} ${imu_cfg["offset_z"]}' rpy='0 0 0'/>
 </joint>
 </robot>

File: rmodus_sim/urdf/imu.urdf.xacro (robot description, xacro)
@@ -2,8 +2,4 @@
 <robot xmlns:xacro='http://www.ros.org/wiki/xacro'
        xmlns:gz='http://gazebosim.org/schema'>
-<!-- PROPERTY -->
-<xacro:property name='imu_offset_z' value='0.015'/>
-<xacro:property name='imu_offset_x' value='0.056'/>
-<xacro:property name='imu_offset_y' value='0.020'/>
 <!-- IMU -->
 <link name='imu_mount'>
@@ -16,5 +12,5 @@
   <parent link='nav_module_mount'/>
   <child link='imu_mount'/>
-  <origin xyz='${imu_offset_x} ${imu_offset_y} ${imu_offset_z}' rpy='0 0 0'/>
+  <origin xyz='${imu_cfg["offset_x"]} ${imu_cfg["offset_y"]} ${imu_cfg["offset_z"]}' rpy='0 0 0'/>
 </joint>
 <gazebo>

File: rmodus_sim/urdf/lidar.urdf.xacro (robot description, xacro)
@@ -2,7 +2,4 @@
 <robot xmlns:xacro='http://www.ros.org/wiki/xacro'
        xmlns:gz='http://gazebosim.org/schema'>
-<!-- PROPERTY -->
-<xacro:property name='lidar_offset_z' value='0.2'/>
-<xacro:property name='lidar_offset_x' value='0.005'/>
 <!-- LIDAR -->
 <link name='lidar_beam'>
@@ -15,5 +12,5 @@
   <parent link='nav_module_mount'/>
   <child link='lidar_beam'/>
-  <origin xyz='${lidar_offset_x} 0 ${lidar_offset_z}' rpy='0 0 0'/>
+  <origin xyz='${lidar_cfg["offset_x"]} 0 ${lidar_cfg["offset_z"]}' rpy='0 0 0'/>
 </joint>
 <gazebo>
