Commit message: autonomy -> localization, navigation

File: rmodus_description/urdf/imu.urdf.xacro (robot description, xacro)
@@ -1,4 +1,4 @@
 <?xml version='1.0'?>
-<!-- Shared IMU TF frame - no Gazebo plugins -->
+<!-- Shared IMU TF frame - no Gazebo plugins. Included only when imu.enabled. -->
 <robot xmlns:xacro='http://www.ros.org/wiki/xacro'>
 <xacro:property name='imu_size' value='${imu_cfg.get("size", [0.02, 0.02, 0.01])}'/>
@@ -29,5 +29,5 @@
 </link>
 <joint name='imu_mount_joint' type='fixed'>
-  <parent link='${imu_cfg.get("mount_parent_frame", "main_module_mount")}'/>
+  <parent link='${imu_cfg.get("mount_parent_frame", "rmodus_mount")}'/>
   <child link='imu_mount'/>
   <origin xyz='${imu_cfg.get("mount_offset", [0.0, 0.0, 0.0])[0]} ${imu_cfg.get("mount_offset", [0.0, 0.0, 0.0])[1]} ${imu_cfg.get("mount_offset", [0.0, 0.0, 0.0])[2]}'

File: rmodus_description/urdf/lidar.urdf.xacro (robot description, xacro)
@@ -1,4 +1,4 @@
 <?xml version='1.0'?>
-<!-- Shared lidar TF frame - no Gazebo plugins -->
+<!-- Shared lidar TF frame - no Gazebo plugins. Included only when lidar.enabled. -->
 <robot xmlns:xacro='http://www.ros.org/wiki/xacro'>
 <xacro:property name='lidar_size' value='${lidar_cfg.get("size", [0.02, 0.02])}'/>
@@ -28,5 +28,5 @@
 </link>
 <joint name='lidar_mount_joint' type='fixed'>
-  <parent link='${lidar_cfg.get("mount_parent_frame", "main_module_mount")}'/>
+  <parent link='${lidar_cfg.get("mount_parent_frame", "rmodus_mount")}'/>
   <child link='lidar_mount'/>
   <origin xyz='${lidar_cfg.get("mount_offset", [0.0, 0.0, 0.0])[0]} ${lidar_cfg.get("mount_offset", [0.0, 0.0, 0.0])[1]} ${lidar_cfg.get("mount_offset", [0.0, 0.0, 0.0])[2]}'

File: rmodus_description/urdf/robot.urdf.xacro (robot description, xacro)
@@ -1,44 +1,29 @@
 <?xml version='1.0'?>
-<!-- Shared robot description entry point.
-     Includes all base URDF components common to both hw and sim.
-     Gazebo plugins are added by rmodus_gazebo/urdf/ includes. -->
+<!-- Kit overlay: rmodus_mount (+ optional imu/lidar) on existing base_link. -->
 <robot
-  name='my_robot'
+  name='rmodus_kit'
   xmlns:xacro='http://www.ros.org/wiki/xacro'>
-<!-- ARGUMENTS -->
 <xacro:arg name='config_path' default='' />
-<!-- CONFIG -->
-<xacro:property name='robot_cfg'     value="${xacro.load_yaml('$(arg config_path)')}" />
-<xacro:property name='base_cfg'      value="${robot_cfg['/**']['ros__parameters']['base_link']}" />
-<xacro:property name='imu_cfg'       value="${robot_cfg['/**']['ros__parameters']['imu']}" />
-<xacro:property name='lidar_cfg'     value="${robot_cfg['/**']['ros__parameters']['lidar']}" />
-<xacro:property name='use_mesh'      value='false' />
-<xacro:property name='meshes_dir'    value='rmodus_description/meshes' />
-<xacro:property name='mesh_scale'    value='1.0' />
-<!-- COLORS -->
+<xacro:arg name='include_chassis' default='false' />
+<xacro:arg name='chassis_contents_path' default='' />
+<xacro:property name='robot_cfg' value="${xacro.load_yaml('$(arg config_path)')}" />
+<xacro:property name='params' value="${robot_cfg['/**']['ros__parameters']}" />
+<xacro:property name='module_cfg' value="${params.get('rmodus_module', params.get('nav_module', dict()))}" />
+<xacro:property name='imu_cfg' value="${params.get('imu', dict())}" />
+<xacro:property name='lidar_cfg' value="${params.get('lidar', dict())}" />
+<xacro:property name='use_mesh' value='false' />
+<xacro:property name='meshes_dir' value='rmodus_description/meshes' />
+<xacro:property name='mesh_scale' value='1.0' />
 <xacro:property name='alpha' value='1'/>
-<xacro:property name='base_color' value='0.28 0.31 0.35 ${alpha}'/>
 <xacro:property name='main_module_color' value='0.45 0.48 0.52 ${alpha}'/>
-<xacro:property name='wheel_color' value='0.20 0.22 0.24 ${alpha}'/>
 <xacro:property name='imu_mount_color' value='1.0 0.62 0.20 ${alpha}'/>
 <xacro:property name='imu_link_color' value='1.0 0.82 0.35 ${alpha}'/>
 <xacro:property name='lidar_mount_color' value='0.30 0.62 1.0 ${alpha}'/>
 <xacro:property name='lidar_beam_color' value='0.10 0.90 0.95 ${alpha}'/>
-<xacro:property name='bumper_mount_color' value='0.90 0.78 0.12 ${alpha}'/>
-<xacro:property name='bumper_contact_color' value='1.0 0.95 0.25 ${alpha}'/>
-<xacro:property name='cliff_mount_color' value='0.78 0.35 0.88 ${alpha}'/>
-<xacro:property name='cliff_beam_color' value='0.95 0.45 1.0 ${alpha}'/>
-<material name='base_mat'> <color rgba='${base_color}'/> </material>
 <material name='main_module_mat'> <color rgba='${main_module_color}'/> </material>
-<material name='wheel_mat'> <color rgba='${wheel_color}'/> </material>
 <material name='imu_mount_mat'> <color rgba='${imu_mount_color}'/> </material>
 <material name='imu_link_mat'> <color rgba='${imu_link_color}'/> </material>
 <material name='lidar_mount_mat'> <color rgba='${lidar_mount_color}'/> </material>
 <material name='lidar_beam_mat'> <color rgba='${lidar_beam_color}'/> </material>
-<material name='bumper_mount_mat'> <color rgba='${bumper_mount_color}'/> </material>
-<material name='bumper_contact_mat'> <color rgba='${bumper_contact_color}'/> </material>
-<material name='cliff_mount_mat'> <color rgba='${cliff_mount_color}'/> </material>
-<material name='cliff_beam_mat'> <color rgba='${cliff_beam_color}'/> </material>
-<!-- INERTIA HELPERS -->
 <xacro:macro name='box_inertia' params='m x y z'>
   <inertial>
@@ -49,24 +34,20 @@
   </inertial>
 </xacro:macro>
-<xacro:macro name='cylinder_inertia' params='m r h'>
-  <inertial>
-    <mass value='${m}'/>
-    <inertia ixx='${m/12 * (3*r*r + h*h)}' ixy='0.0' ixz='0.0'
-             iyy='${m/12 * (3*r*r + h*h)}' iyz='0.0'
-             izz='${m/2 * r*r}'/>
-  </inertial>
-</xacro:macro>
-<xacro:macro name='sphere_inertia' params='m r'>
-  <inertial>
-    <mass value='${m}'/>
-    <inertia ixx='${2/5 * m * r * r}' ixy='0.0' ixz='0.0'
-             iyy='${2/5 * m * r * r}' iyz='0.0'
-             izz='${2/5 * m * r * r}'/>
-  </inertial>
-</xacro:macro>
-<!-- INCLUDES: box + optional lidar/imu TF frames.
-     Bumper / cliff TF are published by rmodus_bumper / rmodus_cliff_sensor launches. -->
-<xacro:include filename='base.urdf.xacro'/>
-<xacro:include filename='imu.urdf.xacro'/>
-<xacro:include filename='lidar.urdf.xacro'/>
+<!-- Host: either compose rmodus_chassis or stub base_link for foreign platform. -->
+<xacro:if value="$(arg include_chassis)">
+  <xacro:property name='base_cfg' value="${params['base_link']}" />
+  <xacro:include filename="$(arg chassis_contents_path)"/>
+  <xacro:rmodus_chassis_links/>
+</xacro:if>
+<xacro:unless value="$(arg include_chassis)">
+  <!-- Reference link only; foreign host (or prior RSP) owns base_link TF. -->
+  <link name='base_link'/>
+</xacro:unless>
+<xacro:include filename='rmodus_module.urdf.xacro'/>
+<xacro:if value="${imu_cfg.get('enabled', False)}">
+  <xacro:include filename='imu.urdf.xacro'/>
+</xacro:if>
+<xacro:if value="${lidar_cfg.get('enabled', False)}">
+  <xacro:include filename='lidar.urdf.xacro'/>
+</xacro:if>
 </robot>
