Commit message: splitting ros2 packages + estop

File: rmodus_description/urdf/robot.urdf.xacro (robot description, xacro)
@@ -10,6 +10,4 @@
 <!-- CONFIG -->
 <xacro:property name='robot_cfg'     value="${xacro.load_yaml('$(arg config_path)')}" />
-<xacro:property name='bumpers'       value="${robot_cfg['/**']['ros__parameters']['bumpers']}" />
-<xacro:property name='cliff_sensors' value="${robot_cfg['/**']['ros__parameters']['cliff_sensors']}" />
 <xacro:property name='base_cfg'      value="${robot_cfg['/**']['ros__parameters']['base_link']}" />
 <xacro:property name='imu_cfg'       value="${robot_cfg['/**']['ros__parameters']['imu']}" />
@@ -67,9 +65,8 @@
   </inertial>
 </xacro:macro>
-<!-- INCLUDES -->
+<!-- INCLUDES: box + optional lidar/imu TF frames.
+     Bumper / cliff TF are published by rmodus_bumper / rmodus_cliff_sensor launches. -->
 <xacro:include filename='base.urdf.xacro'/>
 <xacro:include filename='imu.urdf.xacro'/>
 <xacro:include filename='lidar.urdf.xacro'/>
-<xacro:include filename='bumpers.urdf.xacro'/>
-<xacro:include filename='cliff_sensors.urdf.xacro'/>
 </robot>

File: rmodus_sim/urdf/robot.urdf.xacro (robot description, xacro)
@@ -17,6 +17,7 @@
 <!-- Shared config and helpers -->
 <xacro:property name='robot_cfg' value="${xacro.load_yaml('$(arg config_path)')}" />
-<xacro:property name='bumpers' value="${robot_cfg['/**']['ros__parameters']['bumpers']}" />
-<xacro:property name='cliff_sensors' value="${robot_cfg['/**']['ros__parameters']['cliff_sensors']}" />
+<!-- bumpers/cliff: list (legacy) or {items: [...]} (module config) -->
+<xacro:property name='bumpers' value="${(lambda b: (b.get('items', []) if isinstance(b, dict) else (b or [])))(robot_cfg['/**']['ros__parameters'].get('bumpers', []))}" />
+<xacro:property name='cliff_sensors' value="${(lambda c: (c.get('items', []) if isinstance(c, dict) else (c or [])))(robot_cfg['/**']['ros__parameters'].get('cliff_sensors', []))}" />
 <xacro:property name='base_cfg' value="${robot_cfg['/**']['ros__parameters']['base_link']}" />
 <xacro:property name='imu_cfg' value="${robot_cfg['/**']['ros__parameters']['imu']}" />

Commit message: sim->gazbeo rename

File: rmodus_description/urdf/robot.urdf.xacro (robot description, xacro)
@@ -2,5 +2,5 @@
 <!-- Shared robot description entry point.
      Includes all base URDF components common to both hw and sim.
-     Gazebo plugins are added by rmodus_sim/urdf/ includes. -->
+     Gazebo plugins are added by rmodus_gazebo/urdf/ includes. -->
 <robot
   name='my_robot'

File: rmodus_gazebo/urdf/robot.urdf.xacro (robot description, xacro)
@@ -13,5 +13,5 @@
 <xacro:property name='use_mesh' value='$(arg use_mesh_visuals)' />
 <!-- CONSTANTS used by sim-specific xacro (mesh paths) -->
-<xacro:property name='meshes_dir' value='rmodus_sim/meshes'/>
+<xacro:property name='meshes_dir' value='rmodus_gazebo/meshes'/>
 <xacro:property name='creo_scale' value='0.001' />
 <!-- Shared config and helpers -->

Commit message: sjednoceni generovani modelu robota

File: rmodus_description/urdf/robot.urdf.xacro (robot description, xacro)
@@ -1,22 +1,35 @@
 <?xml version='1.0'?>
-<!-- Kit overlay: rmodus_mount (+ optional imu/lidar) on existing base_link. -->
+<!-- One robot model for the real machine and for Gazebo.
+     joint_type=fixed on the robot (wheel TF without /joint_states).
+     joint_type=continuous in sim so the drive plugin can spin the wheels.
+     gazebo_overlay includes rmodus_gazebo plugins; it does not add geometry. -->
 <robot
-  name='rmodus_kit'
-  xmlns:xacro='http://www.ros.org/wiki/xacro'>
-<xacro:arg name='config_path' default='' />
-<xacro:arg name='include_chassis' default='false' />
-<xacro:arg name='chassis_contents_path' default='' />
-<xacro:property name='robot_cfg' value="${xacro.load_yaml('$(arg config_path)')}" />
-<xacro:property name='params' value="${robot_cfg['/**']['ros__parameters']}" />
-<xacro:property name='module_cfg' value="${params.get('rmodus_module', params.get('nav_module', dict()))}" />
-<xacro:property name='imu_cfg' value="${params.get('imu', dict())}" />
-<xacro:property name='lidar_cfg' value="${params.get('lidar', dict())}" />
-<xacro:property name='bumpers_cfg' value="${params.get('bumpers', dict())}" />
-<xacro:property name='bumper_items' value="${bumpers_cfg.get('items', []) if bumpers_cfg.get('enabled', False) else []}" />
-<xacro:property name='parts_cfg' value="${params.get('parts', dict())}" />
-<xacro:property name='part_items' value="${parts_cfg.get('items', []) if parts_cfg.get('enabled', True) else []}" />
-<xacro:property name='use_mesh' value='false' />
-<xacro:property name='meshes_dir' value='rmodus_description/meshes' />
-<xacro:property name='mesh_scale' value='1.0' />
+  name='rmodus'
+  xmlns:xacro='http://www.ros.org/wiki/xacro'
+  xmlns:gz='http://gazebosim.org/schema'>
+<xacro:arg name='config_path' default=''/>
+<xacro:arg name='include_chassis' default='false'/>
+<xacro:arg name='chassis_contents_path' default=''/>
+<xacro:arg name='joint_type' default='fixed'/>
+<xacro:arg name='gazebo_overlay' default='false'/>
+<xacro:arg name='gazebo_urdf_dir' default=''/>
+<xacro:property name='robot_cfg' value="${xacro.load_yaml('$(arg config_path)')}"/>
+<xacro:property name='params' value="${robot_cfg['/**']['ros__parameters']}"/>
+<xacro:property name='module_cfg' value="${params.get('rmodus_module', params.get('nav_module', dict()))}"/>
+<xacro:property name='imu_cfg' value="${params.get('imu', dict())}"/>
+<xacro:property name='lidar_cfg' value="${params.get('lidar', dict())}"/>
+<xacro:property name='bumpers_cfg' value="${params.get('bumpers', dict())}"/>
+<xacro:property name='bumper_items' value="${bumpers_cfg.get('items', []) if bumpers_cfg.get('enabled', False) else []}"/>
+<xacro:property name='bumpers' value="${[b for b in bumper_items if b.get('enabled', True)]}"/>
+<xacro:property name='parts_cfg' value="${params.get('parts', dict())}"/>
+<xacro:property name='part_items' value="${parts_cfg.get('items', []) if parts_cfg.get('enabled', True) else []}"/>
+<xacro:property name='cliffs_cfg' value="${params.get('cliff_sensors', dict())}"/>
+<xacro:property name='cliff_sensors' value="${[c for c in (cliffs_cfg.get('items') or []) if c.get('enabled', True)] if cliffs_cfg.get('enabled', False) else []}"/>
+<xacro:property name='imu_on' value='${bool(imu_cfg.get("enabled", False))}'/>
+<xacro:property name='lidar_on' value='${bool(lidar_cfg.get("enabled", False))}'/>
+<xacro:property name='cliffs_on' value='${bool(cliff_sensors)}'/>
+<xacro:property name='use_mesh' value='false'/>
+<xacro:property name='meshes_dir' value='rmodus_description/meshes'/>
+<xacro:property name='mesh_scale' value='1.0'/>
 <xacro:property name='alpha' value='1'/>
 <xacro:property name='main_module_color' value='0.45 0.48 0.52 ${alpha}'/>
@@ -26,4 +39,5 @@
 <xacro:property name='lidar_beam_color' value='0.10 0.90 0.95 ${alpha}'/>
 <xacro:property name='bumper_mount_color' value='0.68 0.20 0.20 ${alpha}'/>
+<xacro:property name='cliff_mount_color' value='0.18 0.62 0.44 ${alpha}'/>
 <material name='main_module_mat'> <color rgba='${main_module_color}'/> </material>
 <material name='imu_mount_mat'> <color rgba='${imu_mount_color}'/> </material>
@@ -32,4 +46,5 @@
 <material name='lidar_beam_mat'> <color rgba='${lidar_beam_color}'/> </material>
 <material name='bumper_mount_mat'> <color rgba='${bumper_mount_color}'/> </material>
+<material name='cliff_mount_mat'> <color rgba='${cliff_mount_color}'/> </material>
 <xacro:macro name='box_inertia' params='m x y z'>
   <inertial>
@@ -40,23 +55,42 @@
   </inertial>
 </xacro:macro>
-<!-- Host: either compose rmodus_chassis or stub base_link for foreign platform. -->
+<!-- Host: rmodus_chassis, or a stub base_link when a foreign platform already publishes it. -->
 <xacro:if value="$(arg include_chassis)">
-  <xacro:property name='base_cfg' value="${params['base_link']}" />
-  <xacro:property name='drive_cfg' value="${params.get('drive', dict())}" />
+  <xacro:property name='base_cfg' value="${params['base_link']}"/>
+  <xacro:property name='drive_cfg' value="${params.get('drive', dict())}"/>
   <xacro:include filename="$(arg chassis_contents_path)"/>
-  <xacro:rmodus_chassis_links/>
+  <xacro:rmodus_chassis_links joint_type='$(arg joint_type)'/>
 </xacro:if>
 <xacro:unless value="$(arg include_chassis)">
-  <!-- Reference link only; foreign host (or prior RSP) owns base_link TF. -->
   <link name='base_link'/>
 </xacro:unless>
 <xacro:include filename='rmodus_module.urdf.xacro'/>
-<xacro:if value="${imu_cfg.get('enabled', False)}">
+<xacro:if value='${imu_on}'>
   <xacro:include filename='imu.urdf.xacro'/>
 </xacro:if>
-<xacro:if value="${lidar_cfg.get('enabled', False)}">
+<xacro:if value='${lidar_on}'>
   <xacro:include filename='lidar.urdf.xacro'/>
 </xacro:if>
 <xacro:include filename='bumper_bodies.urdf.xacro'/>
 <xacro:include filename='parts.urdf.xacro'/>
+<xacro:if value='${cliffs_on}'>
+  <xacro:include filename='cliff_sensors.urdf.xacro'/>
+</xacro:if>
+<!-- Plugins only. Paths come from the sim launch so this package does not require rmodus_gazebo. -->
+<xacro:if value="$(arg gazebo_overlay)">
+  <xacro:if value='${lidar_on or cliffs_on}'>
+    <xacro:include filename='$(arg gazebo_urdf_dir)/gz_sensors.urdf.xacro'/>
+  </xacro:if>
+  <xacro:if value='${imu_on}'>
+    <xacro:include filename='$(arg gazebo_urdf_dir)/gz_imu.urdf.xacro'/>
+  </xacro:if>
+  <xacro:if value='${lidar_on}'>
+    <xacro:include filename='$(arg gazebo_urdf_dir)/gz_lidar.urdf.xacro'/>
+  </xacro:if>
+  <xacro:include filename='$(arg gazebo_urdf_dir)/gz_bumpers.urdf.xacro'/>
+  <xacro:if value='${cliffs_on}'>
+    <xacro:include filename='$(arg gazebo_urdf_dir)/gz_cliff_sensors.urdf.xacro'/>
+  </xacro:if>
+  <xacro:include filename='$(arg gazebo_urdf_dir)/control.urdf.xacro'/>
+</xacro:if>
 </robot>

File: rmodus_gazebo/urdf/robot.urdf.xacro (robot description, xacro)
@@ -1,7 +1,5 @@
 <?xml version='1.0'?>
-<!-- Sim twin of the real robot.
-     Geometry comes from the same profile YAML and the same xacro fragments
-     as rmodus_chassis + rmodus_description. This file only adds Gazebo plugins
-     and continuous wheel joints so /cmd_vel can drive the model. -->
+<!-- Sim defaults for the single model in rmodus_description/urdf/robot.urdf.xacro.
+     Geometry is not copied here. Launch passes the same arguments directly. -->
 <robot
   name='rmodus'
@@ -10,72 +8,8 @@
 <xacro:arg name='config_path' default=''/>
 <xacro:arg name='chassis_contents_path' default='$(find rmodus_chassis)/urdf/chassis_contents.urdf.xacro'/>
-<xacro:arg name='description_urdf_dir' default='$(find rmodus_description)/urdf'/>
-<xacro:property name='robot_cfg' value="${xacro.load_yaml('$(arg config_path)')}"/>
-<xacro:property name='params' value="${robot_cfg['/**']['ros__parameters']}"/>
-<xacro:property name='base_cfg' value="${params['base_link']}"/>
-<xacro:property name='drive_cfg' value="${params.get('drive', dict())}"/>
-<xacro:property name='module_cfg' value="${params.get('rmodus_module', params.get('nav_module', dict()))}"/>
-<xacro:property name='imu_cfg' value="${params.get('imu', dict())}"/>
-<xacro:property name='lidar_cfg' value="${params.get('lidar', dict())}"/>
-<xacro:property name='bumpers_cfg' value="${params.get('bumpers', dict())}"/>
-<xacro:property name='bumper_items' value="${bumpers_cfg.get('items', []) if bumpers_cfg.get('enabled', False) else []}"/>
-<xacro:property name='bumpers' value="${[b for b in bumper_items if b.get('enabled', True)]}"/>
-<xacro:property name='parts_cfg' value="${params.get('parts', dict())}"/>
-<xacro:property name='part_items' value="${parts_cfg.get('items', []) if parts_cfg.get('enabled', True) else []}"/>
-<xacro:property name='cliffs_cfg' value="${params.get('cliff_sensors', dict())}"/>
-<xacro:property name='cliff_sensors' value="${[c for c in (cliffs_cfg.get('items') or []) if c.get('enabled', True)] if cliffs_cfg.get('enabled', False) else []}"/>
-<xacro:property name='imu_on' value='${bool(imu_cfg.get("enabled", False))}'/>
-<xacro:property name='lidar_on' value='${bool(lidar_cfg.get("enabled", False))}'/>
-<xacro:property name='cliffs_on' value='${bool(cliff_sensors)}'/>
-<xacro:property name='alpha' value='1'/>
-<xacro:property name='main_module_color' value='0.45 0.48 0.52 ${alpha}'/>
-<xacro:property name='imu_mount_color' value='1.0 0.62 0.20 ${alpha}'/>
-<xacro:property name='imu_link_color' value='1.0 0.82 0.35 ${alpha}'/>
-<xacro:property name='lidar_mount_color' value='0.30 0.62 1.0 ${alpha}'/>
-<xacro:property name='lidar_beam_color' value='0.10 0.90 0.95 ${alpha}'/>
-<xacro:property name='bumper_mount_color' value='0.68 0.20 0.20 ${alpha}'/>
-<xacro:property name='cliff_mount_color' value='0.18 0.62 0.44 ${alpha}'/>
-<material name='main_module_mat'> <color rgba='${main_module_color}'/> </material>
-<material name='imu_mount_mat'> <color rgba='${imu_mount_color}'/> </material>
-<material name='imu_link_mat'> <color rgba='${imu_link_color}'/> </material>
-<material name='lidar_mount_mat'> <color rgba='${lidar_mount_color}'/> </material>
-<material name='lidar_beam_mat'> <color rgba='${lidar_beam_color}'/> </material>
-<material name='bumper_mount_mat'> <color rgba='${bumper_mount_color}'/> </material>
-<material name='cliff_mount_mat'> <color rgba='${cliff_mount_color}'/> </material>
-<xacro:macro name='box_inertia' params='m x y z'>
-  <inertial>
-    <mass value='${m}'/>
-    <inertia ixx='${m/12 * (y*y + z*z)}' ixy='0.0' ixz='0.0'
-             iyy='${m/12 * (x*x + z*z)}' iyz='0.0'
-             izz='${m/12 * (x*x + y*y)}'/>
-  </inertial>
-</xacro:macro>
-<xacro:include filename='$(arg chassis_contents_path)'/>
-<xacro:rmodus_chassis_links joint_type='continuous'/>
-<xacro:include filename='$(arg description_urdf_dir)/rmodus_module.urdf.xacro'/>
-<xacro:if value='${imu_on}'>
-  <xacro:include filename='$(arg description_urdf_dir)/imu.urdf.xacro'/>
-</xacro:if>
-<xacro:if value='${lidar_on}'>
-  <xacro:include filename='$(arg description_urdf_dir)/lidar.urdf.xacro'/>
-</xacro:if>
-<xacro:include filename='$(arg description_urdf_dir)/bumper_bodies.urdf.xacro'/>
-<xacro:include filename='$(arg description_urdf_dir)/parts.urdf.xacro'/>
-<xacro:if value='${cliffs_on}'>
-  <xacro:include filename='$(arg description_urdf_dir)/cliff_sensors.urdf.xacro'/>
-</xacro:if>
-<xacro:if value='${lidar_on or cliffs_on}'>
-  <xacro:include filename='gz_sensors.urdf.xacro'/>
-</xacro:if>
-<xacro:if value='${imu_on}'>
-  <xacro:include filename='gz_imu.urdf.xacro'/>
-</xacro:if>
-<xacro:if value='${lidar_on}'>
-  <xacro:include filename='gz_lidar.urdf.xacro'/>
-</xacro:if>
-<xacro:include filename='gz_bumpers.urdf.xacro'/>
-<xacro:if value='${cliffs_on}'>
-  <xacro:include filename='gz_cliff_sensors.urdf.xacro'/>
-</xacro:if>
-<xacro:include filename='control.urdf.xacro'/>
+<xacro:arg name='include_chassis' default='true'/>
+<xacro:arg name='joint_type' default='continuous'/>
+<xacro:arg name='gazebo_overlay' default='true'/>
+<xacro:arg name='gazebo_urdf_dir' default='$(find rmodus_gazebo)/urdf'/>
+<xacro:include filename='$(find rmodus_description)/urdf/robot.urdf.xacro'/>
 </robot>
