Commit message: frames prefixes remove

File: rmodus_description/urdf/bumper_bodies.urdf.xacro (robot description, xacro)
@@ -1,7 +1,8 @@
 <?xml version='1.0'?>
-<!-- Bumpers: bumper_<name>_mount = physical box centred on mount_offset,
-     frame_id (default bumper_<name>_contact) = contact point, by default on the front face [size[0]/2, 0, 0].
+<!-- Bumper: <name>_mount = box centred on mount_offset,
+     frame_id (default <name>_contact) = contact, by default on the front face [size[0]/2, 0, 0].
+     Collision is named <name>_mount; sdformat appends _collision itself.
      rmodus_bumper publishes the same chain as static TF only when description is not running.
-     Expects bumper_items in scope. -->
+     Expects bumper_items in scope. name is the whole stem (front or bumper_front). -->
 <robot xmlns:xacro='http://www.ros.org/wiki/xacro'>
 <xacro:macro name='render_bumper_body' params='b'>
@@ -12,6 +13,6 @@
     <xacro:property name='coff' value='${b.get("contact_offset", [bsize[0] / 2.0, 0.0, 0.0])}'/>
     <xacro:property name='crpy' value='${b.get("contact_rpy", [0.0, 0.0, 0.0])}'/>
-    <xacro:property name='cframe' value='${b.get("frame_id") or "bumper_" + b["name"] + "_contact"}'/>
-    <link name='bumper_${b["name"]}_mount'>
+    <xacro:property name='cframe' value='${b.get("frame_id") or b["name"] + "_contact"}'/>
+    <link name='${b["name"]}_mount'>
       <inertial>
         <mass value='0.01'/>
@@ -22,11 +23,11 @@
         <material name='bumper_mount_mat'/>
       </visual>
-      <collision name='bumper_${b["name"]}_mount_collision'>
+      <collision name='${b["name"]}_mount'>
         <geometry><box size='${bsize[0]} ${bsize[1]} ${bsize[2]}'/></geometry>
       </collision>
     </link>
-    <joint name='bumper_${b["name"]}_mount_joint' type='fixed'>
+    <joint name='${b["name"]}_mount_joint' type='fixed'>
       <parent link='${b.get("mount_parent_frame", "base_link")}'/>
-      <child link='bumper_${b["name"]}_mount'/>
+      <child link='${b["name"]}_mount'/>
       <origin xyz='${boff[0]} ${boff[1]} ${boff[2]}' rpy='${brpy[0]} ${brpy[1]} ${brpy[2]}'/>
     </joint>
@@ -37,6 +38,6 @@
       </inertial>
     </link>
-    <joint name='bumper_${b["name"]}_contact_joint' type='fixed'>
-      <parent link='bumper_${b["name"]}_mount'/>
+    <joint name='${b["name"]}_contact_joint' type='fixed'>
+      <parent link='${b["name"]}_mount'/>
       <child link='${cframe}'/>
       <origin xyz='${coff[0]} ${coff[1]} ${coff[2]}' rpy='${crpy[0]} ${crpy[1]} ${crpy[2]}'/>

File: rmodus_description/urdf/cliff_sensors.urdf.xacro (robot description, xacro)
@@ -1,8 +1,11 @@
 <?xml version='1.0'?>
-<!-- Shared cliff sensor TF frames - no Gazebo plugins -->
+<!-- Cliff: <name>_mount = box, beam link = frame_id or <name>_beam.
+     Same expression as rmodus_cliff_sensor launch (Range header and static TF).
+     name is the whole stem (fl or cliff_sensor_fl). -->
 <robot xmlns:xacro='http://www.ros.org/wiki/xacro'>
 <xacro:property name='cliff_sensor_mass' value='0.001'/>
 <xacro:macro name='render_cliff_sensor' params='c'>
-  <link name='cliff_sensor_${c["name"]}_mount'>
+  <xacro:property name='cframe' value='${c.get("frame_id") or c["name"] + "_beam"}'/>
+  <link name='${c["name"]}_mount'>
     <xacro:box_inertia m='${cliff_sensor_mass}' x='${c["size"][0]}' y='${c["size"][1]}' z='${c["size"][2]}'/>
     <visual>
@@ -11,16 +14,16 @@
       <material name='cliff_mount_mat'/>
     </visual>
-    <collision>
+    <collision name='${c["name"]}_mount'>
       <origin xyz='${c["size"][0]/2} 0 ${-c["size"][2]/2}' rpy='0 0 0'/>
       <geometry><box size='${c["size"][0]} ${c["size"][1]} ${c["size"][2]}'/></geometry>
     </collision>
   </link>
-  <joint name='cliff_sensor_${c["name"]}_mount_joint' type='fixed'>
+  <joint name='${c["name"]}_mount_joint' type='fixed'>
     <parent link='${c.get("mount_parent_frame", c.get("parent_frame", "base_link"))}'/>
-    <child link='cliff_sensor_${c["name"]}_mount'/>
+    <child link='${c["name"]}_mount'/>
     <origin xyz='${c.get("mount_offset", c.get("offset", [0.0, 0.0, 0.0]))[0]} ${c.get("mount_offset", c.get("offset", [0.0, 0.0, 0.0]))[1]} ${c.get("mount_offset", c.get("offset", [0.0, 0.0, 0.0]))[2]}'
             rpy='${c.get("mount_rpy", [0.0, 0.0, c.get("yaw", 0.0)])[0]} ${c.get("mount_rpy", [0.0, 0.0, c.get("yaw", 0.0)])[1]} ${c.get("mount_rpy", [0.0, 0.0, c.get("yaw", 0.0)])[2]}'/>
   </joint>
-  <link name='cliff_sensor_${c["name"]}_beam'>
+  <link name='${cframe}'>
     <inertial>
       <mass value='0.001'/>
@@ -28,7 +31,7 @@
     </inertial>
   </link>
-  <joint name='cliff_sensor_${c["name"]}_beam_joint' type='fixed'>
-    <parent link='cliff_sensor_${c["name"]}_mount'/>
-    <child link='cliff_sensor_${c["name"]}_beam'/>
+  <joint name='${c["name"]}_beam_joint' type='fixed'>
+    <parent link='${c["name"]}_mount'/>
+    <child link='${cframe}'/>
     <origin xyz='${c.get("beam_offset", [c["size"][0], 0.0, -c["size"][2]/2])[0]} ${c.get("beam_offset", [c["size"][0], 0.0, -c["size"][2]/2])[1]} ${c.get("beam_offset", [c["size"][0], 0.0, -c["size"][2]/2])[2]}'
             rpy='${c.get("beam_rpy", [0.0, pi/2, 0.0])[0]} ${c.get("beam_rpy", [0.0, pi/2, 0.0])[1]} ${c.get("beam_rpy", [0.0, pi/2, 0.0])[2]}'/>

File: rmodus_gazebo/urdf/gz_bumpers.urdf.xacro (robot description, xacro)
@@ -1,22 +1,25 @@
 <?xml version='1.0'?>
-<!-- Contact sensors on bumper_<name>_mount. The world already loads Contact.
-     GZ topic is internal; sim_bumper_bridge republishes UInt8MultiArray
-     on bumpers.state_topic. rmodus_bumper turns that into Bumper. -->
+<!-- Contact sensor <name>_sensor on link <name>_mount. The world already loads Contact.
+     Harmonic publishes
+     /world/my_world/model/rmodus/link/<name>_mount/sensor/<name>_sensor/contact.
+     The bridge maps that onto /sim/bumper/<name>/contact.
+     URDF collision is named <name>_mount; the filter uses <name>_mount_collision
+     because sdformat appends _collision itself. -->
 <robot xmlns:xacro='http://www.ros.org/wiki/xacro'>
 <xacro:macro name='gz_bumper_sensors' params='b'>
   <xacro:if value='${b.get("enabled", True)}'>
-    <gazebo reference='bumper_${b["name"]}_mount_joint'>
+    <gazebo reference='${b["name"]}_mount_joint'>
       <preserveFixedJoint>true</preserveFixedJoint>
     </gazebo>
-    <gazebo reference='bumper_${b["name"]}_contact_joint'>
+    <gazebo reference='${b["name"]}_contact_joint'>
       <preserveFixedJoint>true</preserveFixedJoint>
     </gazebo>
-    <gazebo reference='bumper_${b["name"]}_mount'>
-      <sensor name='bumper_${b["name"]}_sensor' type='contact'>
+    <gazebo reference='${b["name"]}_mount'>
+      <sensor name='${b["name"]}_sensor' type='contact'>
         <always_on>1</always_on>
         <update_rate>${b.get("update_rate", 30)}</update_rate>
         <topic>/sim/bumper/${b["name"]}/contact</topic>
         <contact>
-          <collision>bumper_${b["name"]}_mount_collision</collision>
+          <collision>${b["name"]}_mount_collision</collision>
         </contact>
       </sensor>

File: rmodus_gazebo/urdf/gz_cliff_sensors.urdf.xacro (robot description, xacro)
@@ -1,22 +1,24 @@
 <?xml version='1.0'?>
-<!-- Downward ray on cliff_sensor_<name>_beam.
-     Publishes LaserScan on an internal topic; sim_cliff_bridge packs meters
-     into cliff_sensors.state_topic. rmodus_cliff_sensor turns that into Range. -->
+<!-- Ray <name>_ray on the beam link: frame_id, or <name>_beam.
+     Publishes LaserScan on /sim/cliff/<name>/scan; sim_cliff_bridge packs meters
+     into cliff_sensors.state_topic. rmodus_cliff_sensor turns that into Range.
+     name is the whole stem (fl or cliff_sensor_fl). -->
 <robot xmlns:xacro='http://www.ros.org/wiki/xacro'>
 <xacro:macro name='gz_cliff_sensor' params='c'>
   <xacro:if value='${c.get("enabled", True)}'>
-    <gazebo reference='cliff_sensor_${c["name"]}_mount_joint'>
+    <xacro:property name='cframe' value='${c.get("frame_id") or c["name"] + "_beam"}'/>
+    <gazebo reference='${c["name"]}_mount_joint'>
       <preserveFixedJoint>true</preserveFixedJoint>
     </gazebo>
-    <gazebo reference='cliff_sensor_${c["name"]}_beam_joint'>
+    <gazebo reference='${c["name"]}_beam_joint'>
       <preserveFixedJoint>true</preserveFixedJoint>
     </gazebo>
-    <gazebo reference='cliff_sensor_${c["name"]}_beam'>
-      <sensor name='cliff_${c["name"]}' type='gpu_ray'>
+    <gazebo reference='${cframe}'>
+      <sensor name='${c["name"]}_ray' type='gpu_ray'>
         <always_on>1</always_on>
         <update_rate>${c.get("update_rate", 20)}</update_rate>
         <visualize>${str(c.get("visualize", False)).lower()}</visualize>
         <topic>/sim/cliff/${c["name"]}/scan</topic>
-        <gz_frame_id>cliff_sensor_${c["name"]}_beam</gz_frame_id>
+        <gz_frame_id>${cframe}</gz_frame_id>
         <ray>
           <scan>
