Commit message: tf working is now

File: rmodus_chassis/urdf/chassis.urdf.xacro (robot description, xacro)
@@ -7,4 +7,5 @@
 <xacro:property name='robot_cfg' value="${xacro.load_yaml('$(arg config_path)')}" />
 <xacro:property name='base_cfg' value="${robot_cfg['/**']['ros__parameters']['base_link']}" />
+<xacro:property name='drive_cfg' value="${robot_cfg['/**']['ros__parameters'].get('drive', dict())}" />
 <xacro:include filename="chassis_contents.urdf.xacro"/>
 <xacro:rmodus_chassis_links/>

File: rmodus_chassis/urdf/chassis_contents.urdf.xacro (robot description, xacro)
@@ -1,4 +1,4 @@
 <?xml version='1.0'?>
-<!-- Host links only (no <robot> wrapper). Expects base_cfg in scope. -->
+<!-- Host links only (no <robot> wrapper). Expects base_cfg and drive_cfg in scope. -->
 <robot xmlns:xacro='http://www.ros.org/wiki/xacro'>
 <xacro:macro name='rmodus_chassis_box_inertia' params='m x y z'>
@@ -34,4 +34,46 @@
     <origin xyz='0 0 ${base_offset_z}' rpy='0 0 0'/>
   </joint>
+  <xacro:rmodus_chassis_wheels/>
+</xacro:macro>
+<!-- Wheel centre z sits wheel_radius above base_footprint. Fixed joints: TF must not wait for /joint_states. -->
+<xacro:macro name='rmodus_chassis_wheel' params='name x y radius width z'>
+  <link name='${name}_link'>
+    <xacro:rmodus_chassis_box_inertia m='0.3' x='${2*radius}' y='${width}' z='${2*radius}'/>
+    <visual>
+      <origin xyz='0 0 0' rpy='${pi/2} 0 0'/>
+      <geometry><cylinder radius='${radius}' length='${width}'/></geometry>
+      <material name='wheel_mat'/>
+    </visual>
+    <collision>
+      <origin xyz='0 0 0' rpy='${pi/2} 0 0'/>
+      <geometry><cylinder radius='${radius}' length='${width}'/></geometry>
+    </collision>
+  </link>
+  <joint name='${name}' type='fixed'>
+    <parent link='base_link'/>
+    <child link='${name}_link'/>
+    <origin xyz='${x} ${y} ${z}' rpy='0 0 0'/>
+  </joint>
+</xacro:macro>
+<xacro:macro name='rmodus_chassis_wheels'>
+  <xacro:property name='wheel_mode' value='${drive_cfg.get("mode", "")}'/>
+  <xacro:property name='wheel_r' value='${float(drive_cfg.get("wheel_radius", 0.05))}'/>
+  <xacro:property name='wheel_w' value='${float(drive_cfg.get("wheel_width", 0.04))}'/>
+  <xacro:property name='wheel_hx' value='${float(drive_cfg.get("wheelbase", 0.0)) / 2.0}'/>
+  <xacro:property name='wheel_hy' value='${float(drive_cfg.get("track_width", 0.3)) / 2.0}'/>
+  <xacro:property name='wheel_z' value='${wheel_r - float(base_cfg["offset_z"])}'/>
+  <material name='wheel_mat'>
+    <color rgba='0.10 0.10 0.11 1'/>
+  </material>
+  <xacro:if value='${wheel_mode in ("mecanum", "diff4")}'>
+    <xacro:rmodus_chassis_wheel name='wheel_fl' x='${wheel_hx}' y='${wheel_hy}' radius='${wheel_r}' width='${wheel_w}' z='${wheel_z}'/>
+    <xacro:rmodus_chassis_wheel name='wheel_fr' x='${wheel_hx}' y='${-wheel_hy}' radius='${wheel_r}' width='${wheel_w}' z='${wheel_z}'/>
+    <xacro:rmodus_chassis_wheel name='wheel_rl' x='${-wheel_hx}' y='${wheel_hy}' radius='${wheel_r}' width='${wheel_w}' z='${wheel_z}'/>
+    <xacro:rmodus_chassis_wheel name='wheel_rr' x='${-wheel_hx}' y='${-wheel_hy}' radius='${wheel_r}' width='${wheel_w}' z='${wheel_z}'/>
+  </xacro:if>
+  <xacro:if value='${wheel_mode == "diff2"}'>
+    <xacro:rmodus_chassis_wheel name='wheel_l' x='0.0' y='${wheel_hy}' radius='${wheel_r}' width='${wheel_w}' z='${wheel_z}'/>
+    <xacro:rmodus_chassis_wheel name='wheel_r' x='0.0' y='${-wheel_hy}' radius='${wheel_r}' width='${wheel_w}' z='${wheel_z}'/>
+  </xacro:if>
 </xacro:macro>
 </robot>

File: rmodus_description/urdf/robot.urdf.xacro (robot description, xacro)
@@ -12,4 +12,8 @@
 <xacro:property name='imu_cfg' value="${params.get('imu', dict())}" />
 <xacro:property name='lidar_cfg' value="${params.get('lidar', dict())}" />
+<xacro:property name='bumpers_cfg' value="${params.get('bumpers', dict())}" />
+<xacro:property name='bumper_items' value="${bumpers_cfg.get('items', []) if bumpers_cfg.get('enabled', False) else []}" />
+<xacro:property name='parts_cfg' value="${params.get('parts', dict())}" />
+<xacro:property name='part_items' value="${parts_cfg.get('items', []) if parts_cfg.get('enabled', True) else []}" />
 <xacro:property name='use_mesh' value='false' />
 <xacro:property name='meshes_dir' value='rmodus_description/meshes' />
@@ -21,4 +25,5 @@
 <xacro:property name='lidar_mount_color' value='0.30 0.62 1.0 ${alpha}'/>
 <xacro:property name='lidar_beam_color' value='0.10 0.90 0.95 ${alpha}'/>
+<xacro:property name='bumper_mount_color' value='0.68 0.20 0.20 ${alpha}'/>
 <material name='main_module_mat'> <color rgba='${main_module_color}'/> </material>
 <material name='imu_mount_mat'> <color rgba='${imu_mount_color}'/> </material>
@@ -26,4 +31,5 @@
 <material name='lidar_mount_mat'> <color rgba='${lidar_mount_color}'/> </material>
 <material name='lidar_beam_mat'> <color rgba='${lidar_beam_color}'/> </material>
+<material name='bumper_mount_mat'> <color rgba='${bumper_mount_color}'/> </material>
 <xacro:macro name='box_inertia' params='m x y z'>
   <inertial>
@@ -37,4 +43,5 @@
 <xacro:if value="$(arg include_chassis)">
   <xacro:property name='base_cfg' value="${params['base_link']}" />
+  <xacro:property name='drive_cfg' value="${params.get('drive', dict())}" />
   <xacro:include filename="$(arg chassis_contents_path)"/>
   <xacro:rmodus_chassis_links/>
@@ -51,3 +58,5 @@
   <xacro:include filename='lidar.urdf.xacro'/>
 </xacro:if>
+<xacro:include filename='bumper_bodies.urdf.xacro'/>
+<xacro:include filename='parts.urdf.xacro'/>
 </robot>
