Commit message: sim repair

File: rmodus_chassis/urdf/chassis_contents.urdf.xacro (robot description, xacro)
@@ -10,5 +10,5 @@
   </inertial>
 </xacro:macro>
-<xacro:macro name='rmodus_chassis_links'>
+<xacro:macro name='rmodus_chassis_links' params='joint_type:=fixed'>
   <xacro:property name='base_mass' value='${base_cfg["mass"]}'/>
   <xacro:property name='base_size_x' value='${base_cfg["size"][0]}'/>
@@ -16,5 +16,10 @@
   <xacro:property name='base_size_z' value='${base_cfg["size"][2]}'/>
   <xacro:property name='base_offset_z' value='${base_cfg["offset_z"]}'/>
-  <link name='base_footprint'/>
+  <link name='base_footprint'>
+    <inertial>
+      <mass value='0.001'/>
+      <inertia ixx='1e-6' ixy='0' ixz='0' iyy='1e-6' iyz='0' izz='1e-6'/>
+    </inertial>
+  </link>
   <link name='base_link'>
     <xacro:rmodus_chassis_box_inertia m='${base_mass}' x='${base_size_x}' y='${base_size_y}' z='${base_size_z}'/>
@@ -34,8 +39,10 @@
     <origin xyz='0 0 ${base_offset_z}' rpy='0 0 0'/>
   </joint>
-  <xacro:rmodus_chassis_wheels/>
+  <xacro:rmodus_chassis_wheels joint_type='${joint_type}'/>
 </xacro:macro>
-<!-- Wheel centre z sits wheel_radius above base_footprint. Fixed joints: TF must not wait for /joint_states. -->
-<xacro:macro name='rmodus_chassis_wheel' params='name x y radius width z'>
+<!-- Wheel centre z sits wheel_radius above base_footprint.
+     HW default joint_type=fixed so TF does not wait for /joint_states.
+     Sim passes joint_type=continuous; axis Y matches the cylinder (visual rpy pi/2 about X). -->
+<xacro:macro name='rmodus_chassis_wheel' params='name x y radius width z joint_type:=fixed'>
   <link name='${name}_link'>
     <xacro:rmodus_chassis_box_inertia m='0.3' x='${2*radius}' y='${width}' z='${2*radius}'/>
@@ -50,11 +57,14 @@
     </collision>
   </link>
-  <joint name='${name}' type='fixed'>
+  <joint name='${name}' type='${joint_type}'>
     <parent link='base_link'/>
     <child link='${name}_link'/>
     <origin xyz='${x} ${y} ${z}' rpy='0 0 0'/>
+    <xacro:if value='${joint_type != "fixed"}'>
+      <axis xyz='0 1 0'/>
+    </xacro:if>
   </joint>
 </xacro:macro>
-<xacro:macro name='rmodus_chassis_wheels'>
+<xacro:macro name='rmodus_chassis_wheels' params='joint_type:=fixed'>
   <xacro:property name='wheel_mode' value='${drive_cfg.get("mode", "")}'/>
   <xacro:property name='wheel_r' value='${float(drive_cfg.get("wheel_radius", 0.05))}'/>
@@ -67,12 +77,12 @@
   </material>
   <xacro:if value='${wheel_mode in ("mecanum", "diff4")}'>
-    <xacro:rmodus_chassis_wheel name='wheel_fl' x='${wheel_hx}' y='${wheel_hy}' radius='${wheel_r}' width='${wheel_w}' z='${wheel_z}'/>
-    <xacro:rmodus_chassis_wheel name='wheel_fr' x='${wheel_hx}' y='${-wheel_hy}' radius='${wheel_r}' width='${wheel_w}' z='${wheel_z}'/>
-    <xacro:rmodus_chassis_wheel name='wheel_rl' x='${-wheel_hx}' y='${wheel_hy}' radius='${wheel_r}' width='${wheel_w}' z='${wheel_z}'/>
-    <xacro:rmodus_chassis_wheel name='wheel_rr' x='${-wheel_hx}' y='${-wheel_hy}' radius='${wheel_r}' width='${wheel_w}' z='${wheel_z}'/>
+    <xacro:rmodus_chassis_wheel name='wheel_fl' x='${wheel_hx}' y='${wheel_hy}' radius='${wheel_r}' width='${wheel_w}' z='${wheel_z}' joint_type='${joint_type}'/>
+    <xacro:rmodus_chassis_wheel name='wheel_fr' x='${wheel_hx}' y='${-wheel_hy}' radius='${wheel_r}' width='${wheel_w}' z='${wheel_z}' joint_type='${joint_type}'/>
+    <xacro:rmodus_chassis_wheel name='wheel_rl' x='${-wheel_hx}' y='${wheel_hy}' radius='${wheel_r}' width='${wheel_w}' z='${wheel_z}' joint_type='${joint_type}'/>
+    <xacro:rmodus_chassis_wheel name='wheel_rr' x='${-wheel_hx}' y='${-wheel_hy}' radius='${wheel_r}' width='${wheel_w}' z='${wheel_z}' joint_type='${joint_type}'/>
   </xacro:if>
   <xacro:if value='${wheel_mode == "diff2"}'>
-    <xacro:rmodus_chassis_wheel name='wheel_l' x='0.0' y='${wheel_hy}' radius='${wheel_r}' width='${wheel_w}' z='${wheel_z}'/>
-    <xacro:rmodus_chassis_wheel name='wheel_r' x='0.0' y='${-wheel_hy}' radius='${wheel_r}' width='${wheel_w}' z='${wheel_z}'/>
+    <xacro:rmodus_chassis_wheel name='wheel_l' x='0.0' y='${wheel_hy}' radius='${wheel_r}' width='${wheel_w}' z='${wheel_z}' joint_type='${joint_type}'/>
+    <xacro:rmodus_chassis_wheel name='wheel_r' x='0.0' y='${-wheel_hy}' radius='${wheel_r}' width='${wheel_w}' z='${wheel_z}' joint_type='${joint_type}'/>
   </xacro:if>
 </xacro:macro>

File: rmodus_description/urdf/bumper_bodies.urdf.xacro (robot description, xacro)
@@ -22,5 +22,5 @@
         <material name='bumper_mount_mat'/>
       </visual>
-      <collision>
+      <collision name='bumper_${b["name"]}_mount_collision'>
         <geometry><box size='${bsize[0]} ${bsize[1]} ${bsize[2]}'/></geometry>
       </collision>
@@ -31,5 +31,10 @@
       <origin xyz='${boff[0]} ${boff[1]} ${boff[2]}' rpy='${brpy[0]} ${brpy[1]} ${brpy[2]}'/>
     </joint>
-    <link name='${cframe}'/>
+    <link name='${cframe}'>
+      <inertial>
+        <mass value='0.001'/>
+        <inertia ixx='1e-7' ixy='0' ixz='0' iyy='1e-7' iyz='0' izz='1e-7'/>
+      </inertial>
+    </link>
     <joint name='bumper_${b["name"]}_contact_joint' type='fixed'>
       <parent link='bumper_${b["name"]}_mount'/>

File: rmodus_description/urdf/parts.urdf.xacro (robot description, xacro)
@@ -12,4 +12,8 @@
     <xacro:property name='prpy' value='${p.get("rpy", [0.0, 0.0, 0.0])}'/>
     <link name='${p["name"]}'>
+      <inertial>
+        <mass value='0.001'/>
+        <inertia ixx='1e-6' ixy='0' ixz='0' iyy='1e-6' iyz='0' izz='1e-6'/>
+      </inertial>
       <xacro:if value='${pshape in ("box", "cylinder")}'>
         <visual>

File: rmodus_description/urdf/rmodus_module.urdf.xacro (robot description, xacro)
@@ -12,5 +12,12 @@
 <xacro:property name='mod_size_y' value='${module_cfg.get("size", [0.20, 0.16, 0.05])[1]}'/>
 <xacro:property name='mod_size_z' value='${module_cfg.get("size", [0.20, 0.16, 0.05])[2]}'/>
+<xacro:property name='mod_mass' value='${module_cfg.get("mass", 2.0)}'/>
 <link name='rmodus_mount'>
+  <inertial>
+    <mass value='${mod_mass}'/>
+    <inertia ixx='${mod_mass/12 * (mod_size_y*mod_size_y + mod_size_z*mod_size_z)}' ixy='0' ixz='0'
+             iyy='${mod_mass/12 * (mod_size_x*mod_size_x + mod_size_z*mod_size_z)}' iyz='0'
+             izz='${mod_mass/12 * (mod_size_x*mod_size_x + mod_size_y*mod_size_y)}'/>
+  </inertial>
   <visual>
     <origin xyz='0 0 0' rpy='0 0 0'/>

File: rmodus_gazebo/urdf/control.urdf.xacro (robot description, xacro)
@@ -1,32 +1,82 @@
-<?xml version="1.0"?>
+<?xml version='1.0'?>
+<!-- Drive + joint states. Joint names match rmodus_chassis (wheel_fl, not *_joint). -->
 <robot xmlns:xacro='http://www.ros.org/wiki/xacro'
        xmlns:gz='http://gazebosim.org/schema'>
-<!-- PROPERTY -->
-<!-- mecanum dont publish odom topic in Gazebo 8.9.0 !!!, use 8.10.0 instead or diff-->
-<xacro:property name='drive_mode' value='${drive_cfg.get("mode", "mecanum")}'/> <!-- mecanum or diff/differential -->
-<!-- JOINT STATE plugin -->
+<xacro:property name='drive_on' value='${bool(drive_cfg.get("enabled", False))}'/>
+<xacro:property name='drive_mode' value='${drive_cfg.get("mode", "")}'/>
+<xacro:property name='wheel_radius' value='${float(drive_cfg.get("wheel_radius", 0.05))}'/>
+<xacro:property name='track_width' value='${float(drive_cfg.get("track_width", 0.3))}'/>
+<xacro:property name='wheelbase' value='${float(drive_cfg.get("wheelbase", 0.0))}'/>
+<xacro:property name='cmd_topic' value='${params.get("cmd_mux", dict()).get("output_topic", "/cmd_vel")}'/>
+<xacro:property name='odom_topic' value='${params.get("wheel_odom", dict()).get("topic", "/odom")}'/>
+<xacro:macro name='mecanum_friction' params='link fdir'>
+  <gazebo reference='${link}'>
+    <collision>
+      <surface>
+        <friction>
+          <ode>
+            <mu>1.1</mu>
+            <mu2>0.15</mu2>
+            <fdir1 gz:expressed_in='base_footprint'>${fdir}</fdir1>
+          </ode>
+        </friction>
+      </surface>
+    </collision>
+  </gazebo>
+</xacro:macro>
+<gazebo reference='body_link_joint'>
+  <preserveFixedJoint>true</preserveFixedJoint>
+</gazebo>
+<gazebo reference='rmodus_mount_joint'>
+  <preserveFixedJoint>true</preserveFixedJoint>
+</gazebo>
 <gazebo>
   <plugin
-    filename="libgz-sim-joint-state-publisher-system.so"
-    name="gz::sim::systems::JointStatePublisher">
-    <topic>/joint_states</topic>
+    filename='libgz-sim-joint-state-publisher-system.so'
+    name='gz::sim::systems::JointStatePublisher'>
+    <topic>joint_states</topic>
   </plugin>
 </gazebo>
-<!-- DIFF DRIVE plugin -->
-<xacro:if value="${drive_mode == 'diff' or drive_mode == 'differential'}">
+<xacro:if value='${drive_on and drive_mode == "mecanum"}'>
   <gazebo>
     <plugin
-      filename="libgz-sim-diff-drive-system.so"
-      name="gz::sim::systems::DiffDrive">
-      <left_joint>front_left_wheel_joint</left_joint>
-      <left_joint>rear_left_wheel_joint</left_joint>
-      <right_joint>front_right_wheel_joint</right_joint>
-      <right_joint>rear_right_wheel_joint</right_joint>
+      filename='libgz-sim-mecanum-drive-system.so'
+      name='gz::sim::systems::MecanumDrive'>
+      <front_left_joint>wheel_fl</front_left_joint>
+      <front_right_joint>wheel_fr</front_right_joint>
+      <back_left_joint>wheel_rl</back_left_joint>
+      <back_right_joint>wheel_rr</back_right_joint>
+      <wheel_separation>${track_width}</wheel_separation>
+      <wheelbase>${wheelbase}</wheelbase>
+      <wheel_radius>${wheel_radius}</wheel_radius>
+      <odom_publish_frequency>30</odom_publish_frequency>
+      <topic>${cmd_topic}</topic>
+      <odom_topic>${odom_topic}</odom_topic>
+      <tf_topic>gz_unused_tf</tf_topic>
+      <frame_id>odom</frame_id>
+      <child_frame_id>base_footprint</child_frame_id>
+    </plugin>
+  </gazebo>
+  <!-- Roller slip directions in the footprint frame (X mecanum). -->
+  <xacro:mecanum_friction link='wheel_fl_link' fdir='1 -1 0'/>
+  <xacro:mecanum_friction link='wheel_fr_link' fdir='1 1 0'/>
+  <xacro:mecanum_friction link='wheel_rl_link' fdir='1 1 0'/>
+  <xacro:mecanum_friction link='wheel_rr_link' fdir='1 -1 0'/>
+</xacro:if>
+<xacro:if value='${drive_on and drive_mode == "diff4"}'>
+  <gazebo>
+    <plugin
+      filename='libgz-sim-diff-drive-system.so'
+      name='gz::sim::systems::DiffDrive'>
+      <left_joint>wheel_fl</left_joint>
+      <left_joint>wheel_rl</left_joint>
+      <right_joint>wheel_fr</right_joint>
+      <right_joint>wheel_rr</right_joint>
       <wheel_separation>${track_width}</wheel_separation>
       <wheel_radius>${wheel_radius}</wheel_radius>
       <odom_publish_frequency>30</odom_publish_frequency>
-      <topic>/cmd_vel</topic>
-      <odom_topic>/odom</odom_topic>
-      <tf_topic>__unused_tf</tf_topic>
+      <topic>${cmd_topic}</topic>
+      <odom_topic>${odom_topic}</odom_topic>
+      <tf_topic>gz_unused_tf</tf_topic>
       <frame_id>odom</frame_id>
       <child_frame_id>base_footprint</child_frame_id>
@@ -34,77 +84,21 @@
   </gazebo>
 </xacro:if>
-<!-- MECANUM DRIVE plugin -->
-<xacro:if value="${drive_mode == 'mecanum'}">
+<xacro:if value='${drive_on and drive_mode == "diff2"}'>
   <gazebo>
     <plugin
-      filename='libgz-sim-mecanum-drive-system.so'
-      name='gz::sim::systems::MecanumDrive'>
-      <front_left_joint>front_left_wheel_joint</front_left_joint>
-      <front_right_joint>front_right_wheel_joint</front_right_joint>
-      <back_left_joint>rear_left_wheel_joint</back_left_joint>
-      <back_right_joint>rear_right_wheel_joint</back_right_joint>
+      filename='libgz-sim-diff-drive-system.so'
+      name='gz::sim::systems::DiffDrive'>
+      <left_joint>wheel_l</left_joint>
+      <right_joint>wheel_r</right_joint>
       <wheel_separation>${track_width}</wheel_separation>
-      <wheelbase>${wheelbase}</wheelbase>
       <wheel_radius>${wheel_radius}</wheel_radius>
       <odom_publish_frequency>30</odom_publish_frequency>
-      <topic>/cmd_vel</topic>
-      <odom_topic>/odom</odom_topic>
-      <tf_topic>__unused_tf</tf_topic>
+      <topic>${cmd_topic}</topic>
+      <odom_topic>${odom_topic}</odom_topic>
+      <tf_topic>gz_unused_tf</tf_topic>
       <frame_id>odom</frame_id>
       <child_frame_id>base_footprint</child_frame_id>
     </plugin>
   </gazebo>
-  <gazebo reference='front_left_wheel'>
-    <collision>
-      <surface>
-        <friction>
-          <ode>
-            <mu>${wheel_mu}</mu>
-            <mu2>${wheel_mu2}</mu2>
-            <fdir1 gz:expressed_in='base_footprint'>1 -1 0</fdir1>
-          </ode>
-        </friction>
-      </surface>
-    </collision>
-  </gazebo>
-  <gazebo reference='front_right_wheel'>
-    <collision>
-      <surface>
-        <friction>
-          <ode>
-            <mu>${wheel_mu}</mu>
-            <mu2>${wheel_mu2}</mu2>
-            <fdir1 gz:expressed_in='base_footprint'>1 1 0</fdir1>
-          </ode>
-        </friction>
-      </surface>
-    </collision>
-  </gazebo>
-  <gazebo reference='rear_left_wheel'>
-    <collision>
-      <surface>
-        <friction>
-          <ode>
-            <mu>${wheel_mu}</mu>
-            <mu2>${wheel_mu2}</mu2>
-            <fdir1 gz:expressed_in='base_footprint'>1 1 0</fdir1>
-          </ode>
-        </friction>
-      </surface>
-    </collision>
-  </gazebo>
-  <gazebo reference='rear_right_wheel'>
-    <collision>
-      <surface>
-        <friction>
-          <ode>
-            <mu>${wheel_mu}</mu>
-            <mu2>${wheel_mu2}</mu2>
-            <fdir1 gz:expressed_in='base_footprint'>1 -1 0</fdir1>
-          </ode>
-        </friction>
-      </surface>
-    </collision>
-  </gazebo>
 </xacro:if>
 </robot>

File: rmodus_gazebo/urdf/gz_bumpers.urdf.xacro (robot description, xacro)
@@ -1,29 +1,25 @@
 <?xml version='1.0'?>
-<!-- Sim-only: Gazebo contact sensor plugins for bumpers.
-     TF links/joints are defined in rmodus_description/urdf/bumpers.urdf.xacro -->
-<robot xmlns:xacro='http://www.ros.org/wiki/xacro'
-       xmlns:gz='http://gazebosim.org/schema'>
-<!-- Contact system plugin (one instance for all bumpers) -->
-<gazebo>
-  <plugin filename='libgz-sim-contact-system.so' name='gz::sim::systems::Contact'/>
-</gazebo>
+<!-- Contact sensors on bumper_<name>_mount. The world already loads Contact.
+     GZ topic is internal; sim_bumper_bridge republishes rmodus_interface/Bumper
+     on the profile topic. -->
+<robot xmlns:xacro='http://www.ros.org/wiki/xacro'>
 <xacro:macro name='gz_bumper_sensors' params='b'>
   <xacro:if value='${b.get("enabled", True)}'>
-  <gazebo reference='bumper_${b["name"]}_mount_joint'>
-    <preserveFixedJoint>true</preserveFixedJoint>
-  </gazebo>
-  <gazebo reference='bumper_${b["name"]}_contact_joint'>
-    <preserveFixedJoint>true</preserveFixedJoint>
-  </gazebo>
-  <gazebo reference='bumper_${b["name"]}_mount'>
-    <sensor name='bumper_${b["name"]}_sensor' type='contact'>
-      <always_on>1</always_on>
-      <update_rate>${b.get("update_rate", 30)}</update_rate>
-      <topic>${b.get("topic", "/bumper/" + b["name"])}</topic>
-      <contact>
-        <collision>bumper_${b["name"]}_mount_collision</collision>
-      </contact>
-    </sensor>
-  </gazebo>
+    <gazebo reference='bumper_${b["name"]}_mount_joint'>
+      <preserveFixedJoint>true</preserveFixedJoint>
+    </gazebo>
+    <gazebo reference='bumper_${b["name"]}_contact_joint'>
+      <preserveFixedJoint>true</preserveFixedJoint>
+    </gazebo>
+    <gazebo reference='bumper_${b["name"]}_mount'>
+      <sensor name='bumper_${b["name"]}_sensor' type='contact'>
+        <always_on>1</always_on>
+        <update_rate>${b.get("update_rate", 30)}</update_rate>
+        <topic>/sim/bumper/${b["name"]}/contact</topic>
+        <contact>
+          <collision>bumper_${b["name"]}_mount_collision</collision>
+        </contact>
+      </sensor>
+    </gazebo>
   </xacro:if>
 </xacro:macro>

File: rmodus_gazebo/urdf/gz_cliff_sensors.urdf.xacro (robot description, xacro)
@@ -1,39 +1,37 @@
 <?xml version='1.0'?>
-<!-- Sim-only: Gazebo ray sensor plugins for cliff sensors.
-     TF links/joints are defined in rmodus_description/urdf/cliff_sensors.urdf.xacro -->
-<robot xmlns:xacro='http://www.ros.org/wiki/xacro'
-       xmlns:gz='http://gazebosim.org/schema'>
+<!-- Downward ray on cliff_sensor_<name>_beam.
+     Publishes LaserScan on an internal topic; sim_cliff_bridge turns it into sensor_msgs/Range. -->
+<robot xmlns:xacro='http://www.ros.org/wiki/xacro'>
 <xacro:macro name='gz_cliff_sensor' params='c'>
   <xacro:if value='${c.get("enabled", True)}'>
-  <gazebo reference='cliff_sensor_${c["name"]}_mount_joint'>
-    <preserveFixedJoint>true</preserveFixedJoint>
-  </gazebo>
-  <gazebo reference='cliff_sensor_${c["name"]}_beam_joint'>
-    <preserveFixedJoint>true</preserveFixedJoint>
-  </gazebo>
-  <gazebo reference='cliff_sensor_${c["name"]}_beam'>
-    <sensor name='cliff_${c["name"]}' type='gpu_ray'>
-      <always_on>1</always_on>
-      <update_rate>${c.get("update_rate", 20)}</update_rate>
-      <visualize>${str(c.get("visualize", True)).lower()}</visualize>
-      <ray>
-        <scan>
-          <horizontal>
-            <samples>1</samples>
-            <resolution>1</resolution>
-            <min_angle>0</min_angle>
-            <max_angle>0</max_angle>
-          </horizontal>
-        </scan>
-        <range>
-          <min>${c.get("range_min", 0.01)}</min>
-          <max>${c.get("range_max", 0.5)}</max>
-          <resolution>${c.get("range_resolution", 0.001)}</resolution>
-        </range>
-      </ray>
-      <topic>${c.get("topic", "/cliff/" + c["name"])}</topic>
-      <gz_frame_id>cliff_sensor_${c["name"]}_beam</gz_frame_id>
-    </sensor>
-  </gazebo>
+    <gazebo reference='cliff_sensor_${c["name"]}_mount_joint'>
+      <preserveFixedJoint>true</preserveFixedJoint>
+    </gazebo>
+    <gazebo reference='cliff_sensor_${c["name"]}_beam_joint'>
+      <preserveFixedJoint>true</preserveFixedJoint>
+    </gazebo>
+    <gazebo reference='cliff_sensor_${c["name"]}_beam'>
+      <sensor name='cliff_${c["name"]}' type='gpu_ray'>
+        <always_on>1</always_on>
+        <update_rate>${c.get("update_rate", 20)}</update_rate>
+        <visualize>${str(c.get("visualize", False)).lower()}</visualize>
+        <topic>/sim/cliff/${c["name"]}/scan</topic>
+        <gz_frame_id>cliff_sensor_${c["name"]}_beam</gz_frame_id>
+        <ray>
+          <scan>
+            <horizontal>
+              <samples>1</samples>
+              <resolution>1</resolution>
+              <min_angle>-0.01</min_angle>
+              <max_angle>0.01</max_angle>
+            </horizontal>
+          </scan>
+          <range>
+            <min>${c.get("range_min", 0.01)}</min>
+            <max>${c.get("range_max", 0.5)}</max>
+          </range>
+        </ray>
+      </sensor>
+    </gazebo>
   </xacro:if>
 </xacro:macro>

File: rmodus_gazebo/urdf/gz_imu.urdf.xacro (robot description, xacro)
@@ -1,12 +1,7 @@
 <?xml version='1.0'?>
-<!-- Sim-only: Gazebo IMU sensor plugin.
-     TF link/joint defined in rmodus_description/urdf/imu.urdf.xacro -->
-<robot xmlns:xacro='http://www.ros.org/wiki/xacro'
-       xmlns:gz='http://gazebosim.org/schema'>
+<!-- IMU on the description frame imu_link. Topic follows imu.topic. -->
+<robot xmlns:xacro='http://www.ros.org/wiki/xacro'>
 <gazebo>
-  <plugin
-    filename='libgz-sim-imu-system.so'
-    name='gz::sim::systems::Imu'>
-  </plugin>
+  <plugin filename='libgz-sim-imu-system.so' name='gz::sim::systems::Imu'/>
 </gazebo>
 <gazebo reference='imu_mount_joint'>
@@ -20,14 +15,6 @@
     <always_on>1</always_on>
     <update_rate>${imu_cfg.get("update_rate", 100)}</update_rate>
-    <visualize>${str(imu_cfg.get("visualize", False)).lower()}</visualize>
     <topic>${imu_cfg.get("topic", "/imu/data")}</topic>
-    <imu>
-      <angular_velocity>
-        <x><noise type='gaussian'><mean>0.0</mean><stddev>1e-4</stddev></noise></x>
-      </angular_velocity>
-      <linear_acceleration>
-        <x><noise type='gaussian'><mean>0.0</mean><stddev>1e-3</stddev></noise></x>
-      </linear_acceleration>
-    </imu>
+    <gz_frame_id>${imu_cfg.get("frame_id", "imu_link")}</gz_frame_id>
   </sensor>
 </gazebo>

File: rmodus_gazebo/urdf/gz_lidar.urdf.xacro (robot description, xacro)
@@ -1,14 +1,6 @@
 <?xml version='1.0'?>
-<!-- Sim-only: Gazebo lidar sensor plugin.
-     TF link/joint defined in rmodus_description/urdf/lidar.urdf.xacro -->
-<robot xmlns:xacro='http://www.ros.org/wiki/xacro'
-       xmlns:gz='http://gazebosim.org/schema'>
-<gazebo>
-  <plugin
-    filename='libgz-sim-sensors-system.so'
-    name='gz::sim::systems::Sensors'>
-    <render_engine>ogre2</render_engine>
-  </plugin>
-</gazebo>
+<!-- GPU lidar on the description frame lidar_beam. Topic follows lidar.topic. -->
+<robot xmlns:xacro='http://www.ros.org/wiki/xacro'>
+<xacro:property name='lidar_samples' value='${max(1, int(round(float(lidar_cfg.get("fov", 360)) / max(float(lidar_cfg.get("resolution", 1.0)), 1e-6))))}'/>
 <gazebo reference='lidar_mount_joint'>
   <preserveFixedJoint>true</preserveFixedJoint>
@@ -22,11 +14,13 @@
     <visualize>${str(lidar_cfg.get("visualize", False)).lower()}</visualize>
     <update_rate>${lidar_cfg.get("update_rate", 10)}</update_rate>
+    <topic>${lidar_cfg.get("topic", "/scan")}</topic>
+    <gz_frame_id>${lidar_cfg.get("frame_id", "lidar_beam")}</gz_frame_id>
     <ray>
       <scan>
         <horizontal>
-          <samples>${max(1, int(round(lidar_cfg.get("fov", 360) / max(lidar_cfg.get("resolution", 1.0), 1e-6))))}</samples>
-          <resolution>1.0</resolution>
+          <samples>${lidar_samples}</samples>
+          <resolution>1</resolution>
           <min_angle>${lidar_cfg.get("angle_min", 0.0)}</min_angle>
-          <max_angle>${lidar_cfg.get("angle_max", 2 * pi)}</max_angle>
+          <max_angle>${lidar_cfg.get("angle_max", 6.28318530718)}</max_angle>
         </horizontal>
       </scan>
@@ -36,6 +30,4 @@
       </range>
     </ray>
-    <topic>${lidar_cfg.get("topic", "/scan")}</topic>
-    <gz_frame_id>lidar_beam</gz_frame_id>
   </sensor>
 </gazebo>
