Commit message: sim repair

File: rmodus_gazebo/urdf/robot.urdf.xacro (robot description, xacro)
@@ -1,52 +1,46 @@
 <?xml version='1.0'?>
-<!-- Simulation robot description.
-     Includes the shared base from rmodus_description and adds Gazebo plugins. -->
+<!-- Sim twin of the real robot.
+     Geometry comes from the same profile YAML and the same xacro fragments
+     as rmodus_chassis + rmodus_description. This file only adds Gazebo plugins
+     and continuous wheel joints so /cmd_vel can drive the model. -->
 <robot
-  name='my_robot'
-  xmlns:xacro='http://ros.org/wiki/xacro'
+  name='rmodus'
+  xmlns:xacro='http://www.ros.org/wiki/xacro'
   xmlns:gz='http://gazebosim.org/schema'>
-<!-- ARGUMENTS -->
-<xacro:arg name='config_path' default='' />
-<xacro:arg name='structure_source' default='local' />
-<xacro:arg name='use_mesh_visuals' default='true' />
-<xacro:property name='structure_source' value='$(arg structure_source)'/>
-<xacro:property name='use_mesh' value='$(arg use_mesh_visuals)' />
-<!-- CONSTANTS used by sim-specific xacro (mesh paths) -->
-<xacro:property name='meshes_dir' value='rmodus_gazebo/meshes'/>
-<xacro:property name='creo_scale' value='0.001' />
-<!-- Shared config and helpers -->
-<xacro:property name='robot_cfg' value="${xacro.load_yaml('$(arg config_path)')}" />
-<!-- bumpers/cliff: list (legacy) or {items: [...]} (module config) -->
-<xacro:property name='bumpers' value="${(lambda b: (b.get('items', []) if isinstance(b, dict) else (b or [])))(robot_cfg['/**']['ros__parameters'].get('bumpers', []))}" />
-<xacro:property name='cliff_sensors' value="${(lambda c: (c.get('items', []) if isinstance(c, dict) else (c or [])))(robot_cfg['/**']['ros__parameters'].get('cliff_sensors', []))}" />
-<xacro:property name='base_cfg' value="${robot_cfg['/**']['ros__parameters']['base_link']}" />
-<xacro:property name='imu_cfg' value="${robot_cfg['/**']['ros__parameters']['imu']}" />
-<xacro:property name='lidar_cfg' value="${robot_cfg['/**']['ros__parameters']['lidar']}" />
-<xacro:property name='drive_cfg' value="${robot_cfg['/**']['ros__parameters'].get('drive', dict())}" />
-<xacro:property name='wheels_cfg' value="${robot_cfg['/**']['ros__parameters'].get('wheels', dict())}" />
-<xacro:property name='visual_colors_cfg' value="${robot_cfg['/**']['ros__parameters'].get('visual_colors', dict())}" />
-<xacro:property name='mesh_scale' value='${creo_scale}' />
-<xacro:property name='base_color' value='${visual_colors_cfg.get("base", [0.16, 0.17, 0.20, 1.0])}'/>
-<xacro:property name='main_module_color' value='${visual_colors_cfg.get("main_module", [0.28, 0.30, 0.34, 1.0])}'/>
-<xacro:property name='wheel_color' value='${visual_colors_cfg.get("wheel", [0.12, 0.12, 0.13, 1.0])}'/>
-<xacro:property name='imu_mount_color' value='${visual_colors_cfg.get("imu_mount", [1.0, 0.35, 0.05, 1.0])}'/>
-<xacro:property name='imu_link_color' value='${visual_colors_cfg.get("imu_link", [1.0, 0.70, 0.15, 1.0])}'/>
-<xacro:property name='lidar_mount_color' value='${visual_colors_cfg.get("lidar_mount", [0.10, 0.45, 1.0, 1.0])}'/>
-<xacro:property name='lidar_beam_color' value='${visual_colors_cfg.get("lidar_beam", [0.0, 1.0, 1.0, 1.0])}'/>
-<xacro:property name='bumper_mount_color' value='${visual_colors_cfg.get("bumper_mount", [0.65, 0.10, 1.0, 1.0])}'/>
-<xacro:property name='bumper_contact_color' value='${visual_colors_cfg.get("bumper_contact", [1.0, 0.0, 0.95, 1.0])}'/>
-<xacro:property name='cliff_mount_color' value='${visual_colors_cfg.get("cliff_mount", [0.0, 0.95, 0.25, 1.0])}'/>
-<xacro:property name='cliff_beam_color' value='${visual_colors_cfg.get("cliff_beam", [0.75, 1.0, 0.0, 1.0])}'/>
-<material name='base_mat'> <color rgba='${base_color[0]} ${base_color[1]} ${base_color[2]} ${base_color[3]}'/> </material>
-<material name='main_module_mat'> <color rgba='${main_module_color[0]} ${main_module_color[1]} ${main_module_color[2]} ${main_module_color[3]}'/> </material>
-<material name='wheel_mat'> <color rgba='${wheel_color[0]} ${wheel_color[1]} ${wheel_color[2]} ${wheel_color[3]}'/> </material>
-<material name='imu_mount_mat'> <color rgba='${imu_mount_color[0]} ${imu_mount_color[1]} ${imu_mount_color[2]} ${imu_mount_color[3]}'/> </material>
-<material name='imu_link_mat'> <color rgba='${imu_link_color[0]} ${imu_link_color[1]} ${imu_link_color[2]} ${imu_link_color[3]}'/> </material>
-<material name='lidar_mount_mat'> <color rgba='${lidar_mount_color[0]} ${lidar_mount_color[1]} ${lidar_mount_color[2]} ${lidar_mount_color[3]}'/> </material>
-<material name='lidar_beam_mat'> <color rgba='${lidar_beam_color[0]} ${lidar_beam_color[1]} ${lidar_beam_color[2]} ${lidar_beam_color[3]}'/> </material>
-<material name='bumper_mount_mat'> <color rgba='${bumper_mount_color[0]} ${bumper_mount_color[1]} ${bumper_mount_color[2]} ${bumper_mount_color[3]}'/> </material>
-<material name='bumper_contact_mat'> <color rgba='${bumper_contact_color[0]} ${bumper_contact_color[1]} ${bumper_contact_color[2]} ${bumper_contact_color[3]}'/> </material>
-<material name='cliff_mount_mat'> <color rgba='${cliff_mount_color[0]} ${cliff_mount_color[1]} ${cliff_mount_color[2]} ${cliff_mount_color[3]}'/> </material>
-<material name='cliff_beam_mat'> <color rgba='${cliff_beam_color[0]} ${cliff_beam_color[1]} ${cliff_beam_color[2]} ${cliff_beam_color[3]}'/> </material>
+<xacro:arg name='config_path' default=''/>
+<xacro:arg name='chassis_contents_path' default='$(find rmodus_chassis)/urdf/chassis_contents.urdf.xacro'/>
+<xacro:arg name='description_urdf_dir' default='$(find rmodus_description)/urdf'/>
+<xacro:property name='robot_cfg' value="${xacro.load_yaml('$(arg config_path)')}"/>
+<xacro:property name='params' value="${robot_cfg['/**']['ros__parameters']}"/>
+<xacro:property name='base_cfg' value="${params['base_link']}"/>
+<xacro:property name='drive_cfg' value="${params.get('drive', dict())}"/>
+<xacro:property name='module_cfg' value="${params.get('rmodus_module', params.get('nav_module', dict()))}"/>
+<xacro:property name='imu_cfg' value="${params.get('imu', dict())}"/>
+<xacro:property name='lidar_cfg' value="${params.get('lidar', dict())}"/>
+<xacro:property name='bumpers_cfg' value="${params.get('bumpers', dict())}"/>
+<xacro:property name='bumper_items' value="${bumpers_cfg.get('items', []) if bumpers_cfg.get('enabled', False) else []}"/>
+<xacro:property name='bumpers' value="${[b for b in bumper_items if b.get('enabled', True)]}"/>
+<xacro:property name='parts_cfg' value="${params.get('parts', dict())}"/>
+<xacro:property name='part_items' value="${parts_cfg.get('items', []) if parts_cfg.get('enabled', True) else []}"/>
+<xacro:property name='cliffs_cfg' value="${params.get('cliff_sensors', dict())}"/>
+<xacro:property name='cliff_sensors' value="${[c for c in (cliffs_cfg.get('items') or []) if c.get('enabled', True)] if cliffs_cfg.get('enabled', False) else []}"/>
+<xacro:property name='imu_on' value='${bool(imu_cfg.get("enabled", False))}'/>
+<xacro:property name='lidar_on' value='${bool(lidar_cfg.get("enabled", False))}'/>
+<xacro:property name='cliffs_on' value='${bool(cliff_sensors)}'/>
+<xacro:property name='alpha' value='1'/>
+<xacro:property name='main_module_color' value='0.45 0.48 0.52 ${alpha}'/>
+<xacro:property name='imu_mount_color' value='1.0 0.62 0.20 ${alpha}'/>
+<xacro:property name='imu_link_color' value='1.0 0.82 0.35 ${alpha}'/>
+<xacro:property name='lidar_mount_color' value='0.30 0.62 1.0 ${alpha}'/>
+<xacro:property name='lidar_beam_color' value='0.10 0.90 0.95 ${alpha}'/>
+<xacro:property name='bumper_mount_color' value='0.68 0.20 0.20 ${alpha}'/>
+<xacro:property name='cliff_mount_color' value='0.18 0.62 0.44 ${alpha}'/>
+<material name='main_module_mat'> <color rgba='${main_module_color}'/> </material>
+<material name='imu_mount_mat'> <color rgba='${imu_mount_color}'/> </material>
+<material name='imu_link_mat'> <color rgba='${imu_link_color}'/> </material>
+<material name='lidar_mount_mat'> <color rgba='${lidar_mount_color}'/> </material>
+<material name='lidar_beam_mat'> <color rgba='${lidar_beam_color}'/> </material>
+<material name='bumper_mount_mat'> <color rgba='${bumper_mount_color}'/> </material>
+<material name='cliff_mount_mat'> <color rgba='${cliff_mount_color}'/> </material>
 <xacro:macro name='box_inertia' params='m x y z'>
   <inertial>
@@ -57,42 +51,31 @@
   </inertial>
 </xacro:macro>
-<xacro:macro name='cylinder_inertia' params='m r h'>
-  <inertial>
-    <mass value='${m}'/>
-    <inertia ixx='${m/12 * (3*r*r + h*h)}' ixy='0.0' ixz='0.0'
-             iyy='${m/12 * (3*r*r + h*h)}' iyz='0.0'
-             izz='${m/2 * r*r}'/>
-  </inertial>
-</xacro:macro>
-<xacro:macro name='sphere_inertia' params='m r'>
-  <inertial>
-    <mass value='${m}'/>
-    <inertia ixx='${2/5 * m * r * r}' ixy='0.0' ixz='0.0'
-             iyy='${2/5 * m * r * r}' iyz='0.0'
-             izz='${2/5 * m * r * r}'/>
-  </inertial>
-</xacro:macro>
-<!-- Structural components are switchable by source. -->
-<xacro:if value='${structure_source == "description"}'>
-  <xacro:include filename='$(find rmodus_description)/urdf/base.urdf.xacro'/>
-  <xacro:include filename='$(find rmodus_description)/urdf/imu.urdf.xacro'/>
-  <xacro:include filename='$(find rmodus_description)/urdf/lidar.urdf.xacro'/>
-  <xacro:include filename='$(find rmodus_description)/urdf/bumpers.urdf.xacro'/>
-  <xacro:include filename='$(find rmodus_description)/urdf/cliff_sensors.urdf.xacro'/>
+<xacro:include filename='$(arg chassis_contents_path)'/>
+<xacro:rmodus_chassis_links joint_type='continuous'/>
+<xacro:include filename='$(arg description_urdf_dir)/rmodus_module.urdf.xacro'/>
+<xacro:if value='${imu_on}'>
+  <xacro:include filename='$(arg description_urdf_dir)/imu.urdf.xacro'/>
 </xacro:if>
-<xacro:unless value='${structure_source == "description"}'>
-  <xacro:include filename='base.urdf.xacro'/>
-  <xacro:include filename='imu.urdf.xacro'/>
-  <xacro:include filename='lidar.urdf.xacro'/>
-  <xacro:include filename='bumpers.urdf.xacro'/>
-  <xacro:include filename='cliff_sensors.urdf.xacro'/>
-</xacro:unless>
-<!-- Sim-only: wheels with mesh visuals -->
-<xacro:include filename='wheels.urdf.xacro'/>
-<!-- Sim-only: Gazebo sensor plugins -->
-<xacro:include filename='gz_imu.urdf.xacro'/>
-<xacro:include filename='gz_lidar.urdf.xacro'/>
+<xacro:if value='${lidar_on}'>
+  <xacro:include filename='$(arg description_urdf_dir)/lidar.urdf.xacro'/>
+</xacro:if>
+<xacro:include filename='$(arg description_urdf_dir)/bumper_bodies.urdf.xacro'/>
+<xacro:include filename='$(arg description_urdf_dir)/parts.urdf.xacro'/>
+<xacro:if value='${cliffs_on}'>
+  <xacro:include filename='$(arg description_urdf_dir)/cliff_sensors.urdf.xacro'/>
+</xacro:if>
+<xacro:if value='${lidar_on or cliffs_on}'>
+  <xacro:include filename='gz_sensors.urdf.xacro'/>
+</xacro:if>
+<xacro:if value='${imu_on}'>
+  <xacro:include filename='gz_imu.urdf.xacro'/>
+</xacro:if>
+<xacro:if value='${lidar_on}'>
+  <xacro:include filename='gz_lidar.urdf.xacro'/>
+</xacro:if>
 <xacro:include filename='gz_bumpers.urdf.xacro'/>
-<xacro:include filename='gz_cliff_sensors.urdf.xacro'/>
+<xacro:if value='${cliffs_on}'>
+  <xacro:include filename='gz_cliff_sensors.urdf.xacro'/>
+</xacro:if>
 <xacro:include filename='control.urdf.xacro'/>
 </robot>
